File: KiCad/IRSensors.sch (KiCad schematic (older format))
At the start: 0 parts

Commit message: Added IMU
Parts:
- added R10, R11, R12, R13, R14, R15, R16, R17, R18, R19, R20, R21, R22, R23, R8, R9: 1k, symbol R
- added R7: 2k2, symbol R
- added U10, U11, U12, U5, U6, U7, U8, U9: GP2Y0E02B, symbol GP2Y0E02B
- added U4: TCA9548APWR, symbol TCA9548APWR
Connections:
- new net: R7.2, U4.3 (~Reset)
- new net GND: U10.3 (GND), U11.3 (GND), U12.3 (GND), U4.1 (A0), U4.12 (GND), U4.2 (A1), U4.21 (A2), U5.3 (GND), U6.3 (GND), U7.3 (GND), U8.3 (GND), U9.3 (GND)
- new net SC0: R9.1, U4.5 (SC0), U5.1 (SCL)
- new net SC1: R11.1, U4.7 (SC1), U6.1 (SCL)
- new net SC2: R13.1, U4.9 (SC2), U7.1 (SCL)
- new net SC3: R15.1, U4.11 (SC3), U8.1 (SCL)
- new net SC4: R17.1, U4.14 (SC4), U9.1 (SCL)
- new net SC5: R19.1, U10.1 (SCL), U4.16 (SC5)
- new net SC6: R21.1, U11.1 (SCL), U4.18 (SC6)
- new net SC7: R23.1, U12.1 (SCL), U4.20 (SC7)
- new net SCL: U4.22 (SCL)
- new net SD0: R8.1, U4.4 (SD0), U5.2 (SDA)
- new net SD1: R10.1, U4.6 (SD1), U6.2 (SDA)
- new net SD2: R12.1, U4.8 (SD2), U7.2 (SDA)
- new net SD3: R14.1, U4.10 (SD3), U8.2 (SDA)
- new net SD4: R16.1, U4.13 (SD4), U9.2 (SDA)
- new net SD5: R18.1, U10.2 (SDA), U4.15 (SD5)
- new net SD6: R20.1, U11.2 (SDA), U4.17 (SD6)
- new net SD7: R22.1, U12.2 (SDA), U4.19 (SD7)
- new net SDA: U4.23 (SDA)
- new net VCC: R10.2, R11.2, R12.2, R13.2, R14.2, R15.2, R16.2, R17.2, R18.2, R19.2, R20.2, R21.2, R22.2, R23.2, R7.1, R8.2, R9.2, U10.4 (VDD), U11.4 (VDD), U12.4 (VDD), U4.24 (VCC), U5.4 (VDD), U6.4 (VDD), U7.4 (VDD), U8.4 (VDD), U9.4 (VDD)

Commit message: Lots of changes
Parts:
- removed U5, U6, U7: GP2Y0E02B, symbol GP2Y0E02B
- added U13, U14, U15: GP2Y0E02B, Connectors_JST:JST_SH_BM04B-SRSS-TB_04x1.00mm_Straight, symbol GP2Y0E02B
- R10: renamed from R9; footprint (none) -> Resistors_SMD:R_0805
- R11: renamed from R10; footprint (none) -> Resistors_SMD:R_0805
- R12: renamed from R11; footprint (none) -> Resistors_SMD:R_0805
- R13: renamed from R12; footprint (none) -> Resistors_SMD:R_0805
- R14: renamed from R13; footprint (none) -> Resistors_SMD:R_0805
- R15: renamed from R14; footprint (none) -> Resistors_SMD:R_0805
- R16: renamed from R15; footprint (none) -> Resistors_SMD:R_0805
- R17: renamed from R16; footprint (none) -> Resistors_SMD:R_0805
- R18: renamed from R17; footprint (none) -> Resistors_SMD:R_0805
- R19: renamed from R18; footprint (none) -> Resistors_SMD:R_0805
- R20: renamed from R19; footprint (none) -> Resistors_SMD:R_0805
- R21: renamed from R20; footprint (none) -> Resistors_SMD:R_0805
- R22: renamed from R21; footprint (none) -> Resistors_SMD:R_0805
- R23: renamed from R22; footprint (none) -> Resistors_SMD:R_0805
- R24: renamed from R23; footprint (none) -> Resistors_SMD:R_0805
- R8: renamed from R7; footprint (none) -> Resistors_SMD:R_0805
- R9: renamed from R8; footprint (none) -> Resistors_SMD:R_0805
- U10, U11, U12, U8, U9: footprint (none) -> Connectors_JST:JST_SH_BM04B-SRSS-TB_04x1.00mm_Straight
- U7: renamed from U4; footprint (none) -> Housings_SSOP:TSSOP-24_4.4x7.8mm_Pitch0.65mm
Connections:
- net GND: now also U13.3 (GND), U14.3 (GND), U15.3 (GND)
- net SC0: now also U8.1 (SCL)
- net SC1: now also U9.1 (SCL)
- net SC2: now also U10.1 (SCL)
- net SC3: now also U11.1 (SCL); no longer U8.1 (SCL)
- net SC4: now also U12.1 (SCL); no longer U9.1 (SCL)
- net SC5: now also U13.1 (SCL); no longer U10.1 (SCL)
- net SC6: now also U14.1 (SCL); no longer U11.1 (SCL)
- net SC7: now also U15.1 (SCL); no longer U12.1 (SCL)
- net SD0: now also U8.2 (SDA)
- net SD1: now also U9.2 (SDA)
- net SD2: now also U10.2 (SDA)
- net SD3: now also U11.2 (SDA); no longer U8.2 (SDA)
- net SD4: now also U12.2 (SDA); no longer U9.2 (SDA)
- net SD5: now also U13.2 (SDA); no longer U10.2 (SDA)
- net SD6: now also U14.2 (SDA); no longer U11.2 (SDA)
- net SD7: now also U15.2 (SDA); no longer U12.2 (SDA)
- net VCC: now also U13.4 (VDD), U14.4 (VDD), U15.4 (VDD)
Other:
- note added: "JST SH connectors, 4 pin, 1mm pitch"
