File: KiCad/FreeIMU.sch (KiCad schematic (older format))
At the start: 0 parts

Commit message: Added IMU
Parts:
- added C?: 10nF, Capacitors_SMD:C_0805, symbol C
- added C?: 0.1uF, Capacitors_SMD:C_0805, symbol C
- added C?: 2.2nF, Capacitors_SMD:C_0805, symbol C
- added C?: 0.22uF, Capacitors_SMD:C_0805, symbol C
- added C?: 4.7uF, Capacitors_SMD:C_0805, symbol C
- added U?: HMC5883, Housings_DFN_QFN:QFN-16-1EP_3x3mm_Pitch0.5mm, symbol HMC5883
- added U?: MPU-6050, Housings_DFN_QFN:QFN-24-1EP_4x4mm_Pitch0.5mm, symbol MPU-6050
Connections:
- new net: C?.2, U?.10 (REGOUT)
- new net: C?.2, U?.20 (CPOUT)
- new net: C?.2, U?.10 (C1)
- new net: C?.2, U?.8 (SETP)
- new net DRDY: U?.15 (DRDY)
- new net FSYNC: U?.11 (FSYNC)
- new net GND: C?.1, C?.1, C?.1, C?.1, U?.1 (CLKIN), U?.11 (GND), U?.18 (GND), U?.9 (AD0), U?.9 (GND)
- new net INT: U?.12 (INT)
- new net MPU_SCL: U?.1 (SCL), U?.7 (AUX_CL)
- new net MPU_SDA: U?.16 (SDA), U?.6 (AUX_DA)
- new net SCL: U?.23 (SCL)
- new net SDA: U?.24 (SDA)
- new net SETC: C?.1, U?.12 (SETC)
- new net VCC: C?.2, U?.13 (VDD), U?.13 (VDDIO), U?.2 (VDD), U?.4 (S1), U?.8 (VLOGIC)
Other:
- note added: "MPU-6050 (Farnell: 186474, QFN-24)\nI2C address: 0x68 / 0x69 (depends on AD0 low or high)"

Commit message: Lots of changes
Parts:
- gave numbers to parts that had none: 7
Connections:
- net SETC: no longer names the net of C7.1, U6.12 (SETC)
Changed lines of the file:
@@
 $Descr A4 11693 8268
 encoding utf-8
-Sheet 2 4
+Sheet 2 3
 Title ""
 Date ""
@@
 VCC
 $Comp
-L C C?
+L C C5
 U 1 1 574C3CF5
 P 2400 3100
-F 0 "C?" H 2425 3200 50  0000 L CNN
+F 0 "C5" H 2425 3200 50  0000 L CNN
 F 1 "10nF" H 2425 3000 50  0000 L CNN
 F 2 "Capacitors_SMD:C_0805" H 2438 2950 50  0001 C CNN
@@
 $EndComp
 $Comp
-L GND #PWR?
+L GND #PWR045
 U 1 1 574C3F70
 P 2400 2850
-F 0 "#PWR?" H 2400 2600 50  0001 C CNN
+F 0 "#PWR045" H 2400 2600 50  0001 C CNN
 F 1 "GND" H 2400 2700 50  0000 C CNN
 F 2 "" H 2400 2850 50  0000 C CNN
@@
 FSYNC
 $Comp
-L GND #PWR?
+L GND #PWR046
 U 1 1 574C4065
 P 2700 3850
-F 0 "#PWR?" H 2700 3600 50  0001 C CNN
+F 0 "#PWR046" H 2700 3600 50  0001 C CNN
 F 1 "GND" H 2700 3700 50  0000 C CNN
 F 2 "" H 2700 3850 50  0000 C CNN
@@
 $EndComp
 $Comp
-L GND #PWR?
+L GND #PWR047
 U 1 1 574C40EB
 P 2800 4750
-F 0 "#PWR?" H 2800 4500 50  0001 C CNN
+F 0 "#PWR047" H 2800 4500 50  0001 C CNN
 F 1 "GND" H 2800 4600 50  0000 C CNN
 F 2 "" H 2800 4750 50  0000 C CNN
@@
 GND
 $Comp
-L C C?
+L C C4
 U 1 1 574C41F0
 P 2150 4300
-F 0 "C?" H 2175 4400 50  0000 L CNN
+F 0 "C4" H 2175 4400 50  0000 L CNN
 F 1 "0.1uF" H 2175 4200 50  0000 L CNN
 F 2 "Capacitors_SMD:C_0805" H 2188 4150 50  0001 C CNN
@@
 $EndComp
 $Comp
-L C C?
+L C C6
 U 1 1 574C457F
 P 2450 4300
-F 0 "C?" H 2475 4400 50  0000 L CNN
+F 0 "C6" H 2475 4400 50  0000 L CNN
 F 1 "2.2nF" H 2475 4200 50  0000 L CNN
 F 2 "Capacitors_SMD:C_0805" H 2488 4150 50  0001 C CNN
@@
 $EndComp
 $Comp
-L GND #PWR?
+L GND #PWR048
 U 1 1 574C4E5A
 P 4250 4000
-F 0 "#PWR?" H 4250 3750 50  0001 C CNN
+F 0 "#PWR048" H 4250 3750 50  0001 C CNN
 F 1 "GND" H 4250 3850 50  0000 C CNN
 F 2 "" H 4250 4000 50  0000 C CNN
@@
 FreeIMU
 $Comp
-L HMC5883 U?
+L HMC5883 U6
 U 1 1 574C57C9
 P 7500 3750
-F 0 "U?" H 8000 3050 60  0000 C CNN
+F 0 "U6" H 8000 3050 60  0000 C CNN
 F 1 "HMC5883" H 7500 3750 60  0000 C CNN
 F 2 "Housings_DFN_QFN:QFN-16-1EP_3x3mm_Pitch0.5mm" H 7500 3750 60  0001 C CNN
@@
 VCC
 $Comp
-L C C?
+L C C7
 U 1 1 574C6C91
 P 7800 5000
-F 0 "C?" H 7825 5100 50  0000 L CNN
+F 0 "C7" H 7825 5100 50  0000 L CNN
 F 1 "0.22uF" H 7825 4900 50  0000 L CNN
 F 2 "Capacitors_SMD:C_0805" H 7838 4850 50  0001 C CNN
@@
 	-1   0    0    1
 $EndComp
-Text Label 8600 3450 0    60   ~ 0
-SETC
-Text Label 7800 5400 0    60   ~ 0
-SETC
-$Comp
-L GND #PWR?
+$Comp
+L GND #PWR049
 U 1 1 574C70FE
 P 9450 4350
-F 0 "#PWR?" H 9450 4100 50  0001 C CNN
+F 0 "#PWR049" H 9450 4100 50  0001 C CNN
 F 1 "GND" H 9450 4200 50  0000 C CNN
 F 2 "" H 9450 4350 50  0000 C CNN
@@
 $EndComp
 $Comp
-L C C?
+L C C8
 U 1 1 574C7189
 P 8850 3850
-F 0 "C?" H 8875 3950 50  0000 L CNN
+F 0 "C8" H 8875 3950 50  0000 L CNN
 F 1 "4.7uF" H 8875 3750 50  0000 L CNN
 F 2 "Capacitors_SMD:C_0805" H 8888 3700 50  0001 C CNN
@@
 	6600 4050 6400 4050
 Wire Wire Line
-	8600 3450 8400 3450
+	8400 3450 9850 3450
 Wire Wire Line
 	7800 4850 7800 4650
@@
 	7800 2850 7800 2700
 $Comp
-L MPU-6050 U?
+L MPU-6050 U5
 U 1 1 574CEE9E
 P 3450 3900
-F 0 "U?" H 3450 3450 60  0000 C CNN
+F 0 "U5" H 3450 3450 60  0000 C CNN
 F 1 "MPU-6050" H 3450 4600 60  0000 C CNN
 F 2 "Housings_DFN_QFN:QFN-24-1EP_4x4mm_Pitch0.5mm" H 3250 3950 60  0001 C CNN
@@
 Text HLabel 4450 3800 2    60   Input ~ 0
 SDA
+Wire Wire Line
+	9850 3450 9850 5400
+Wire Wire Line
+	9850 5400 7800 5400
 $EndSCHEMATC

Commit message: Started on PCB rev 2
Parts:
- C4, C5, C6, C7, C8: footprint Capacitors_SMD:C_0805 -> Capacitors_SMD:C_0603
Changed lines of the file:
@@
 F 0 "C5" H 2425 3200 50  0000 L CNN
 F 1 "10nF" H 2425 3000 50  0000 L CNN
-F 2 "Capacitors_SMD:C_0805" H 2438 2950 50  0001 C CNN
+F 2 "Capacitors_SMD:C_0603" H 2438 2950 50  0001 C CNN
 F 3 "" H 2400 3100 50  0000 C CNN
 	1    2400 3100
@@
 F 0 "C4" H 2175 4400 50  0000 L CNN
 F 1 "0.1uF" H 2175 4200 50  0000 L CNN
-F 2 "Capacitors_SMD:C_0805" H 2188 4150 50  0001 C CNN
+F 2 "Capacitors_SMD:C_0603" H 2188 4150 50  0001 C CNN
 F 3 "" H 2150 4300 50  0000 C CNN
 	1    2150 4300
@@
 F 0 "C6" H 2475 4400 50  0000 L CNN
 F 1 "2.2nF" H 2475 4200 50  0000 L CNN
-F 2 "Capacitors_SMD:C_0805" H 2488 4150 50  0001 C CNN
+F 2 "Capacitors_SMD:C_0603" H 2488 4150 50  0001 C CNN
 F 3 "" H 2450 4300 50  0000 C CNN
 	1    2450 4300
@@
 F 0 "C7" H 7825 5100 50  0000 L CNN
 F 1 "0.22uF" H 7825 4900 50  0000 L CNN
-F 2 "Capacitors_SMD:C_0805" H 7838 4850 50  0001 C CNN
+F 2 "Capacitors_SMD:C_0603" H 7838 4850 50  0001 C CNN
 F 3 "" H 7800 5000 50  0000 C CNN
 	1    7800 5000
@@
 F 0 "C8" H 8875 3950 50  0000 L CNN
 F 1 "4.7uF" H 8875 3750 50  0000 L CNN
-F 2 "Capacitors_SMD:C_0805" H 8888 3700 50  0001 C CNN
+F 2 "Capacitors_SMD:C_0603" H 8888 3700 50  0001 C CNN
 F 3 "" H 8850 3850 50  0000 C CNN
 	1    8850 3850
