File: KiCad/Rev 1/FreeIMU.sch (KiCad schematic (older format))
At the start: 7 parts, among them U5 MPU-6050, U6 HMC5883

Commit message: Started on PCB rev 2
Parts:
- C4, C5, C6, C7, C8: footprint Capacitors_SMD:C_0603 -> Capacitors_SMD:C_0805
Changed lines of the file:
@@
 F 0 "C5" H 2425 3200 50  0000 L CNN
 F 1 "10nF" H 2425 3000 50  0000 L CNN
-F 2 "Capacitors_SMD:C_0603" H 2438 2950 50  0001 C CNN
+F 2 "Capacitors_SMD:C_0805" H 2438 2950 50  0001 C CNN
 F 3 "" H 2400 3100 50  0000 C CNN
 	1    2400 3100
@@
 F 0 "C4" H 2175 4400 50  0000 L CNN
 F 1 "0.1uF" H 2175 4200 50  0000 L CNN
-F 2 "Capacitors_SMD:C_0603" H 2188 4150 50  0001 C CNN
+F 2 "Capacitors_SMD:C_0805" H 2188 4150 50  0001 C CNN
 F 3 "" H 2150 4300 50  0000 C CNN
 	1    2150 4300
@@
 F 0 "C6" H 2475 4400 50  0000 L CNN
 F 1 "2.2nF" H 2475 4200 50  0000 L CNN
-F 2 "Capacitors_SMD:C_0603" H 2488 4150 50  0001 C CNN
+F 2 "Capacitors_SMD:C_0805" H 2488 4150 50  0001 C CNN
 F 3 "" H 2450 4300 50  0000 C CNN
 	1    2450 4300
@@
 F 0 "C7" H 7825 5100 50  0000 L CNN
 F 1 "0.22uF" H 7825 4900 50  0000 L CNN
-F 2 "Capacitors_SMD:C_0603" H 7838 4850 50  0001 C CNN
+F 2 "Capacitors_SMD:C_0805" H 7838 4850 50  0001 C CNN
 F 3 "" H 7800 5000 50  0000 C CNN
 	1    7800 5000
@@
 F 0 "C8" H 8875 3950 50  0000 L CNN
 F 1 "4.7uF" H 8875 3750 50  0000 L CNN
-F 2 "Capacitors_SMD:C_0603" H 8888 3700 50  0001 C CNN
+F 2 "Capacitors_SMD:C_0805" H 8888 3700 50  0001 C CNN
 F 3 "" H 8850 3850 50  0000 C CNN
 	1    8850 3850
