File: KiCad/Rev 1/Ghost.sch (KiCad schematic (older format))
At the start: 33 parts, among them P1 MOTOR, P2 SERVO, P3 START, P4 PWM, P5 RGB, Q1 MMBT3904, SW1 BTN1, U1 INA219, U16 Transmissive_Photo_Interrupter, U17 ESP8266_ESP-12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

Commit message: Started on PCB rev 2
Parts:
- C1, C2, C3, C9: footprint Capacitors_SMD:C_0603 -> Capacitors_SMD:C_0805
- R1, R2, R25, R26, R27, R28, R29, R3, R30, R4, R5, R6, R7: footprint Resistors_SMD:R_0603 -> Resistors_SMD:R_0805
Connections:
- net GND: now also P3.3 (P3); no longer P3.2 (P2)
- net START: now also P3.1 (P1); no longer P3.3 (P3)
- net START_POWER: now also P3.2 (P2); no longer P3.1 (P1)
Other:
- note added: "GHOST rev 1"
- note removed: "GHOST (rev 2)"
Changed lines of the file:
@@
 $EndSheet
 Text Notes 4800 1000 0    197  ~ 39
-GHOST (rev 2)
+GHOST rev 1
 $Comp
 L C C1
@@
 F 0 "C1" H 3325 2350 50  0000 L CNN
 F 1 "0.1-1uF" H 3325 2150 50  0000 L CNN
-F 2 "Capacitors_SMD:C_0603" H 3338 2100 50  0001 C CNN
+F 2 "Capacitors_SMD:C_0805" H 3338 2100 50  0001 C CNN
 F 3 "" H 3300 2250 50  0000 C CNN
 	1    3300 2250
@@
 F 0 "C2" H 7925 2300 50  0000 L CNN
 F 1 "470pF" H 7925 2100 50  0000 L CNN
-F 2 "Capacitors_SMD:C_0603" H 7938 2050 50  0001 C CNN
+F 2 "Capacitors_SMD:C_0805" H 7938 2050 50  0001 C CNN
 F 3 "" H 7900 2200 50  0000 C CNN
 	1    7900 2200
@@
 F 0 "C3" H 8325 2050 50  0000 L CNN
 F 1 "2.2uF" H 8325 1850 50  0000 L CNN
-F 2 "Capacitors_SMD:C_0603" H 8338 1800 50  0001 C CNN
+F 2 "Capacitors_SMD:C_0805" H 8338 1800 50  0001 C CNN
 F 3 "" H 8300 1950 50  0000 C CNN
 	1    8300 1950
@@
 F 0 "R1" V 4430 1750 50  0000 C CNN
 F 1 "0.1ohm" V 4250 1750 50  0000 C CNN
-F 2 "Resistors_SMD:R_0603" V 4280 1750 50  0001 C CNN
+F 2 "Resistors_SMD:R_0805" V 4280 1750 50  0001 C CNN
 F 3 "" H 4350 1750 50  0000 C CNN
 	1    4350 1750
@@
 F 0 "R3" V 6330 4300 50  0000 C CNN
 F 1 "2k2" V 6250 4300 50  0000 C CNN
-F 2 "Resistors_SMD:R_0603" V 6180 4300 50  0001 C CNN
+F 2 "Resistors_SMD:R_0805" V 6180 4300 50  0001 C CNN
 F 3 "" H 6250 4300 50  0000 C CNN
 	1    6250 4300
@@
 F 0 "R2" V 6330 3800 50  0000 C CNN
 F 1 "2k2" V 6250 3800 50  0000 C CNN
-F 2 "Resistors_SMD:R_0603" V 6180 3800 50  0001 C CNN
+F 2 "Resistors_SMD:R_0805" V 6180 3800 50  0001 C CNN
 F 3 "" H 6250 3800 50  0000 C CNN
 	1    6250 3800
@@
 F 0 "R5" V 10180 1300 50  0000 C CNN
 F 1 "100" V 10100 1300 50  0000 C CNN
-F 2 "Resistors_SMD:R_0603" V 10030 1300 50  0001 C CNN
+F 2 "Resistors_SMD:R_0805" V 10030 1300 50  0001 C CNN
 F 3 "" H 10100 1300 50  0000 C CNN
 	1    10100 1300
@@
 F 0 "R7" V 10680 1600 50  0000 C CNN
 F 1 "50" V 10600 1600 50  0000 C CNN
-F 2 "Resistors_SMD:R_0603" V 10530 1600 50  0001 C CNN
+F 2 "Resistors_SMD:R_0805" V 10530 1600 50  0001 C CNN
 F 3 "" H 10600 1600 50  0000 C CNN
 	1    10600 1600
@@
 F 0 "R4" V 9680 1700 50  0000 C CNN
 F 1 "40" V 9600 1700 50  0000 C CNN
-F 2 "Resistors_SMD:R_0603" V 9530 1700 50  0001 C CNN
+F 2 "Resistors_SMD:R_0805" V 9530 1700 50  0001 C CNN
 F 3 "" H 9600 1700 50  0000 C CNN
 	1    9600 1700
@@
 	-1   0    0    -1
 $EndComp
-Text GLabel 1500 4350 2    60   Input ~ 0
+Text GLabel 1450 4150 2    60   Input ~ 0
 START
 $Comp
 L GND #PWR026
 U 1 1 574BC667
-P 1500 4250
-F 0 "#PWR026" H 1500 4000 50  0001 C CNN
-F 1 "GND" H 1500 4100 50  0000 C CNN
-F 2 "" H 1500 4250 50  0000 C CNN
-F 3 "" H 1500 4250 50  0000 C CNN
-	1    1500 4250
+P 1450 4350
+F 0 "#PWR026" H 1450 4100 50  0001 C CNN
+F 1 "GND" H 1450 4200 50  0000 C CNN
+F 2 "" H 1450 4350 50  0000 C CNN
+F 3 "" H 1450 4350 50  0000 C CNN
+	1    1450 4350
 	0    -1   -1   0
 $EndComp
@@
 Wire Wire Line
 	1400 3350 1350 3350
+Wire Wire Line
+	1350 4150 1450 4150
+Wire Wire Line
+	1450 4250 1350 4250
+Wire Wire Line
+	1350 4350 1450 4350
 Text GLabel 3450 3700 0    60   Input ~ 0
 MOTOR
@@
 	3800 2250 3700 2250
 Connection ~ 3700 2350
-Text GLabel 1500 4150 2    60   Input ~ 0
+Text GLabel 1450 4250 2    60   Input ~ 0
 START_POWER
 Text GLabel 3450 4000 0    60   Input ~ 0
@@
 F 0 "R6" V 10680 3800 50  0000 C CNN
 F 1 "220" V 10600 3800 50  0000 C CNN
-F 2 "Resistors_SMD:R_0603" V 10530 3800 50  0001 C CNN
+F 2 "Resistors_SMD:R_0805" V 10530 3800 50  0001 C CNN
 F 3 "" H 10600 3800 50  0000 C CNN
 	1    10600 3800
@@
 F 0 "R27" V 8330 5250 50  0000 C CNN
 F 1 "3k3" V 8250 5250 50  0000 C CNN
-F 2 "Resistors_SMD:R_0603" V 8180 5250 50  0001 C CNN
+F 2 "Resistors_SMD:R_0805" V 8180 5250 50  0001 C CNN
 F 3 "" H 8250 5250 50  0000 C CNN
 	1    8250 5250
@@
 F 0 "C9" H 7475 5400 50  0000 L CNN
 F 1 "100nF" H 7475 5200 50  0000 L CNN
-F 2 "Capacitors_SMD:C_0603" H 7488 5150 50  0001 C CNN
+F 2 "Capacitors_SMD:C_0805" H 7488 5150 50  0001 C CNN
 F 3 "" H 7450 5300 50  0000 C CNN
 	1    7450 5300
@@
 F 0 "R30" V 10230 6050 50  0000 C CNN
 F 1 "3k3" V 10150 6050 50  0000 C CNN
-F 2 "Resistors_SMD:R_0603" V 10080 6050 50  0001 C CNN
+F 2 "Resistors_SMD:R_0805" V 10080 6050 50  0001 C CNN
 F 3 "" H 10150 6050 50  0000 C CNN
 	1    10150 6050
@@
 F 0 "R28" V 10050 5150 50  0000 C CNN
 F 1 "3k3" V 10150 5150 50  0000 C CNN
-F 2 "Resistors_SMD:R_0603" V 10080 5150 50  0001 C CNN
+F 2 "Resistors_SMD:R_0805" V 10080 5150 50  0001 C CNN
 F 3 "" H 10150 5150 50  0000 C CNN
 	1    10150 5150
@@
 F 0 "R29" V 10230 5250 50  0000 C CNN
 F 1 "3k3" V 10150 5250 50  0000 C CNN
-F 2 "Resistors_SMD:R_0603" V 10080 5250 50  0001 C CNN
+F 2 "Resistors_SMD:R_0805" V 10080 5250 50  0001 C CNN
 F 3 "" H 10150 5250 50  0000 C CNN
 	1    10150 5250
@@
 F 0 "R25" V 3730 5650 50  0000 C CNN
 F 1 "270" V 3650 5650 50  0000 C CNN
-F 2 "Resistors_SMD:R_0603" V 3580 5650 50  0001 C CNN
+F 2 "Resistors_SMD:R_0805" V 3580 5650 50  0001 C CNN
 F 3 "" H 3650 5650 50  0000 C CNN
 	1    3650 5650
@@
 F 0 "R26" V 5980 6150 50  0000 C CNN
 F 1 "10k" V 5900 6150 50  0000 C CNN
-F 2 "Resistors_SMD:R_0603" V 5830 6150 50  0001 C CNN
+F 2 "Resistors_SMD:R_0805" V 5830 6150 50  0001 C CNN
 F 3 "" H 5900 6150 50  0000 C CNN
 	1    5900 6150
@@
 	3650 3600 3450 3600
 NoConn ~ 3650 4500
-Wire Wire Line
-	1500 4250 1350 4250
-Wire Wire Line
-	1350 4150 1500 4150
-Wire Wire Line
-	1500 4350 1350 4350
 $EndSCHEMATC
