File: KiCad/Rev 1/IRSensors.sch (KiCad schematic (older format))
At the start: 26 parts, among them U10 GP2Y0E02B, U11 GP2Y0E02B, U12 GP2Y0E02B, U13 GP2Y0E02B, U14 GP2Y0E02B, U15 GP2Y0E02B, U7 TCA9548APWR, U8 GP2Y0E02B, U9 GP2Y0E02B

Commit message: Started on PCB rev 2
Parts:
- R10, R11, R12, R13, R14, R15, R16, R17, R18, R19, R20, R21, R22, R23, R24, R8, R9: footprint Resistors_SMD:R_0603 -> Resistors_SMD:R_0805
Changed lines of the file:
@@
 F 0 "R8" V 2580 3000 50  0000 C CNN
 F 1 "2k2" V 2500 3000 50  0000 C CNN
-F 2 "Resistors_SMD:R_0603" V 2430 3000 50  0001 C CNN
+F 2 "Resistors_SMD:R_0805" V 2430 3000 50  0001 C CNN
 F 3 "" H 2500 3000 50  0000 C CNN
 	1    2500 3000
@@
 F 0 "R9" V 5280 1150 50  0000 C CNN
 F 1 "1k" V 5200 1150 50  0000 C CNN
-F 2 "Resistors_SMD:R_0603" V 5130 1150 50  0001 C CNN
+F 2 "Resistors_SMD:R_0805" V 5130 1150 50  0001 C CNN
 F 3 "" H 5200 1150 50  0000 C CNN
 	1    5200 1150
@@
 F 0 "R10" V 5280 1250 50  0000 C CNN
 F 1 "1k" V 5200 1250 50  0000 C CNN
-F 2 "Resistors_SMD:R_0603" V 5130 1250 50  0001 C CNN
+F 2 "Resistors_SMD:R_0805" V 5130 1250 50  0001 C CNN
 F 3 "" H 5200 1250 50  0000 C CNN
 	1    5200 1250
@@
 F 0 "R11" V 5280 1900 50  0000 C CNN
 F 1 "1k" V 5200 1900 50  0000 C CNN
-F 2 "Resistors_SMD:R_0603" V 5130 1900 50  0001 C CNN
+F 2 "Resistors_SMD:R_0805" V 5130 1900 50  0001 C CNN
 F 3 "" H 5200 1900 50  0000 C CNN
 	1    5200 1900
@@
 F 0 "R12" V 5280 2000 50  0000 C CNN
 F 1 "1k" V 5200 2000 50  0000 C CNN
-F 2 "Resistors_SMD:R_0603" V 5130 2000 50  0001 C CNN
+F 2 "Resistors_SMD:R_0805" V 5130 2000 50  0001 C CNN
 F 3 "" H 5200 2000 50  0000 C CNN
 	1    5200 2000
@@
 F 0 "R13" V 5280 2650 50  0000 C CNN
 F 1 "1k" V 5200 2650 50  0000 C CNN
-F 2 "Resistors_SMD:R_0603" V 5130 2650 50  0001 C CNN
+F 2 "Resistors_SMD:R_0805" V 5130 2650 50  0001 C CNN
 F 3 "" H 5200 2650 50  0000 C CNN
 	1    5200 2650
@@
 F 0 "R14" V 5280 2750 50  0000 C CNN
 F 1 "1k" V 5200 2750 50  0000 C CNN
-F 2 "Resistors_SMD:R_0603" V 5130 2750 50  0001 C CNN
+F 2 "Resistors_SMD:R_0805" V 5130 2750 50  0001 C CNN
 F 3 "" H 5200 2750 50  0000 C CNN
 	1    5200 2750
@@
 F 0 "R15" V 5280 3400 50  0000 C CNN
 F 1 "1k" V 5200 3400 50  0000 C CNN
-F 2 "Resistors_SMD:R_0603" V 5130 3400 50  0001 C CNN
+F 2 "Resistors_SMD:R_0805" V 5130 3400 50  0001 C CNN
 F 3 "" H 5200 3400 50  0000 C CNN
 	1    5200 3400
@@
 F 0 "R16" V 5280 3500 50  0000 C CNN
 F 1 "1k" V 5200 3500 50  0000 C CNN
-F 2 "Resistors_SMD:R_0603" V 5130 3500 50  0001 C CNN
+F 2 "Resistors_SMD:R_0805" V 5130 3500 50  0001 C CNN
 F 3 "" H 5200 3500 50  0000 C CNN
 	1    5200 3500
@@
 F 0 "R17" V 5280 4150 50  0000 C CNN
 F 1 "1k" V 5200 4150 50  0000 C CNN
-F 2 "Resistors_SMD:R_0603" V 5130 4150 50  0001 C CNN
+F 2 "Resistors_SMD:R_0805" V 5130 4150 50  0001 C CNN
 F 3 "" H 5200 4150 50  0000 C CNN
 	1    5200 4150
@@
 F 0 "R18" V 5280 4250 50  0000 C CNN
 F 1 "1k" V 5200 4250 50  0000 C CNN
-F 2 "Resistors_SMD:R_0603" V 5130 4250 50  0001 C CNN
+F 2 "Resistors_SMD:R_0805" V 5130 4250 50  0001 C CNN
 F 3 "" H 5200 4250 50  0000 C CNN
 	1    5200 4250
@@
 F 0 "R19" V 5280 4900 50  0000 C CNN
 F 1 "1k" V 5200 4900 50  0000 C CNN
-F 2 "Resistors_SMD:R_0603" V 5130 4900 50  0001 C CNN
+F 2 "Resistors_SMD:R_0805" V 5130 4900 50  0001 C CNN
 F 3 "" H 5200 4900 50  0000 C CNN
 	1    5200 4900
@@
 F 0 "R20" V 5280 5000 50  0000 C CNN
 F 1 "1k" V 5200 5000 50  0000 C CNN
-F 2 "Resistors_SMD:R_0603" V 5130 5000 50  0001 C CNN
+F 2 "Resistors_SMD:R_0805" V 5130 5000 50  0001 C CNN
 F 3 "" H 5200 5000 50  0000 C CNN
 	1    5200 5000
@@
 F 0 "R21" V 5280 5650 50  0000 C CNN
 F 1 "1k" V 5200 5650 50  0000 C CNN
-F 2 "Resistors_SMD:R_0603" V 5130 5650 50  0001 C CNN
+F 2 "Resistors_SMD:R_0805" V 5130 5650 50  0001 C CNN
 F 3 "" H 5200 5650 50  0000 C CNN
 	1    5200 5650
@@
 F 0 "R22" V 5280 5750 50  0000 C CNN
 F 1 "1k" V 5200 5750 50  0000 C CNN
-F 2 "Resistors_SMD:R_0603" V 5130 5750 50  0001 C CNN
+F 2 "Resistors_SMD:R_0805" V 5130 5750 50  0001 C CNN
 F 3 "" H 5200 5750 50  0000 C CNN
 	1    5200 5750
@@
 F 0 "R23" V 5280 6400 50  0000 C CNN
 F 1 "1k" V 5200 6400 50  0000 C CNN
-F 2 "Resistors_SMD:R_0603" V 5130 6400 50  0001 C CNN
+F 2 "Resistors_SMD:R_0805" V 5130 6400 50  0001 C CNN
 F 3 "" H 5200 6400 50  0000 C CNN
 	1    5200 6400
@@
 F 0 "R24" V 5280 6500 50  0000 C CNN
 F 1 "1k" V 5200 6500 50  0000 C CNN
-F 2 "Resistors_SMD:R_0603" V 5130 6500 50  0001 C CNN
+F 2 "Resistors_SMD:R_0805" V 5130 6500 50  0001 C CNN
 F 3 "" H 5200 6500 50  0000 C CNN
 	1    5200 6500
