File: KiCad/GhostSensorboard/FreeIMU.sch (KiCad schematic (older format))
At the start: 7 parts, among them U5 MPU-6050, U6 HMC5883

Commit message: Routing finished. Playing around with BOM as XSL file.
Parts:
- U6: footprint Housings_DFN_QFN:QFN-16-1EP_3x3mm_Pitch0.5mm -> NorBotKiCadFootprints:HMC5883
Changed lines of the file:
@@
 LIBS:switches
 LIBS:GhostSensorboard-cache
-EELAYER 25 0
+EELAYER 26 0
 EELAYER END
 $Descr A4 11693 8268
 encoding utf-8
 Sheet 2 2
-Title ""
-Date ""
-Rev ""
-Comp ""
+Title "Ghost Sensorboard"
+Date "2017-02-25"
+Rev "1"
+Comp "Frode Lillerud"
 Comment1 ""
 Comment2 ""
@@
 F 0 "U6" H 8000 3050 60  0000 C CNN
 F 1 "HMC5883" H 7500 3750 60  0000 C CNN
-F 2 "Housings_DFN_QFN:QFN-16-1EP_3x3mm_Pitch0.5mm" H 7500 3750 60  0001 C CNN
+F 2 "NorBotKiCadFootprints:HMC5883" H 7500 3750 60  0001 C CNN
 F 3 "" H 7500 3750 60  0000 C CNN
 	1    7500 3750

Commit message: Both boards done, and sent to Elecrow.
Other:
- note added: "HMC5883 compass\nFarnell no: 197-1743\nI2C address: 0x1E"
- note added: "MPU-6050 gyro/accelerometer\nFarnellno: 186-474\nFootprint: QFN-24\nI2C address: 0x68 / 0x69 (depends on AD0 low or high)"
- note removed: "MPU-6050 (Farnell: 186474, QFN-24)\nI2C address: 0x68 / 0x69 (depends on AD0 low or high)"
Changed lines of the file:
@@
 Comment4 ""
 $EndDescr
-Text Notes 2700 2150 0    60   ~ 0
-MPU-6050 (Farnell: 186474, QFN-24)\nI2C address: 0x68 / 0x69 (depends on AD0 low or high)
+Text Notes 2900 2750 0    60   ~ 0
+MPU-6050 gyro/accelerometer\nFarnellno: 186-474\nFootprint: QFN-24\nI2C address: 0x68 / 0x69 (depends on AD0 low or high)
 Text HLabel 2000 3400 0    60   Input ~ 0
 VCC
@@
 Wire Wire Line
 	9850 5400 7800 5400
+Text Notes 8550 2800 0    60   ~ 0
+HMC5883 compass\nFarnell no: 197-1743\nI2C address: 0x1E
 $EndSCHEMATC
