File: KiCad/GhostSensorboard/GhostSensorboard.sch (KiCad schematic (older format))
At the start: 37 parts, among them P1 StartModule, P2 SteeringServo, P3 SteeringServo, P4 CONN_02X30, Q1 BSS138, Q2 BSS138, SW1 SW_Push, U1 TCA9548ARGER, U10 GP2Y0E02B, U11 GP2Y0E02B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

Commit message: GhostESP32 and GhostSensorboard mostly done - but with wrong 60 pin connector
Parts:
- removed RN3, RN4: R_Pack04, symbol R_Pack04
- added RN5: R_Pack08, Resistors_SMD:R_Array_Convex_8x0602, symbol R_Pack08
- C1, C2, C3: footprint (none) -> Capacitors_SMD:C_0603
- D1: footprint (none) -> LEDs:LED_0805
- P1, P2: footprint (none) -> Pin_Headers:Pin_Header_Straight_1x03_Pitch2.54mm
- P3: value SteeringServo -> Motor; footprint (none) -> Pin_Headers:Pin_Header_Straight_1x03_Pitch2.54mm
- P4: footprint (none) -> hrs-fx8c:hrs-fx8c-60p-sv
- R1, R10, R11, R2, R3, R4, R5, R6, R7, R8, R9: footprint (none) -> Resistors_SMD:R_0603_HandSoldering
- RN1, RN2: footprint (none) -> Resistors_SMD:R_Array_Convex_4x0603
- SW1: footprint (none) -> Buttons_Switches_SMD:SW_SPST_EVQP2
- U1: footprint (none) -> Housings_DFN_QFN:QFN-24_4x4mm_Pitch0.5mm
- U10, U11, U12, U2, U3, U7, U8, U9: footprint (none) -> Connectors_JST:JST_SH_BM04B-SRSS-TB_04x1.00mm_Straight
- U13: footprint (none) -> SMD_Packages:SOIC-8-N
- U4: footprint (none) -> NorBotKiCadFootprints:TSOP75x
Connections:
- net +3V3: now also P4.2 (P2), P4.4 (P4), RN5.10 (R7.2), RN5.11 (R6.2), RN5.12 (R5.2), RN5.13 (R4.2), RN5.14 (R3.2), RN5.15 (R2.2), RN5.16 (R1.2), RN5.9 (R8.2); no longer P4.1 (P1)
- net +5V: now also P4.20 (P20), P4.21 (P21), P4.22 (P22), P4.23 (P23), P4.24 (P24), P4.7 (P7), P4.9 (P9); no longer P4.10 (P10), P4.2 (P2), P4.4 (P4), P4.6 (P6)
- net GND: now also P4.11 (P11), P4.13 (P13), P4.15 (P15), P4.26 (P26), P4.27 (P27), P4.28 (P28), P4.29 (P29), P4.30 (P30), P4.41 (P41); no longer P4.35 (P35), P4.37 (P37), P4.39 (P39), P4.7 (P7), P4.9 (P9)
- net GPIO_BUTTON: now also P4.48 (P48); no longer P4.25 (P25)
- net GPIO_DRDY: now also P4.58 (P58); no longer P4.22 (P22)
- net GPIO_FSYNC: now also P4.39 (P39); no longer P4.26 (P26)
- net GPIO_INT: now also P4.37 (P37); no longer P4.24 (P24)
- net GPIO_IR: now also P4.1 (P1); no longer P4.29 (P29)
- net GPIO_LED: now also P4.57 (P57); no longer P4.27 (P27)
- net GPIO_MOTOR: now also P4.60 (P60); no longer P4.13 (P13)
- net GPIO_SCL: now also P4.51 (P51); no longer P4.19 (P19)
- net GPIO_SDA: now also P4.52 (P52); no longer P4.17 (P17)
- net GPIO_STEERING: now also P4.59 (P59); no longer P4.15 (P15)
- net GPIO_StartModule: now also P4.53 (P53); no longer P4.21 (P21)
- net SC0: now also RN1.3 (R3.1); no longer RN1.2 (R2.1), U10.1 (SCL), U11.1 (SCL), U12.1 (SCL), U3.1 (SCL), U7.1 (SCL), U8.1 (SCL), U9.1 (SCL)
- net SC1: now also RN1.1 (R1.1), U3.1 (SCL); no longer RN1.4 (R4.1)
- net SC2: now also RN2.3 (R3.1), U7.1 (SCL); no longer RN2.2 (R2.1)
- net SC3: now also RN2.1 (R1.1), U8.1 (SCL); no longer RN2.4 (R4.1)
- net SC4: now also U9.1 (SCL), RN5.7 (R7.1)
- net SC5: now also U10.1 (SCL), RN5.5 (R5.1)
- net SC6: now also U11.1 (SCL), RN5.3 (R3.1)
- net SC7: now also U12.1 (SCL), RN5.1 (R1.1)
- net SD0: now also RN1.4 (R4.1); no longer RN1.1 (R1.1), U10.2 (SDA), U11.2 (SDA), U12.2 (SDA), U3.2 (SDA), U7.2 (SDA), U8.2 (SDA), U9.2 (SDA)
- net SD1: now also RN1.2 (R2.1), U3.2 (SDA); no longer RN1.3 (R3.1)
- net SD2: now also RN2.4 (R4.1), U7.2 (SDA); no longer RN2.1 (R1.1)
- net SD3: now also RN2.2 (R2.1), U8.2 (SDA); no longer RN2.3 (R3.1)
- net SD4: now also U9.2 (SDA), RN5.8 (R8.1)
- net SD5: now also U10.2 (SDA), RN5.6 (R6.1)
- net SD6: now also U11.2 (SDA), RN5.4 (R4.1)
- net SD7: now also U12.2 (SDA), RN5.2 (R2.1)
- no-connect marks 30 -> 23
Other:
- note added: "Infrared Receiver, 38kHz\n(May optionally replace StartModule)\nTSOP75538WTR, Farnell no: 225-1430 (or similar)\nVoltage: 2.5-5.5V"
- note added: "Pull-up resistors for the IR-sensors\n4 x 1k ohm resistor network.\nFarnell no: 923-4519\n8 x 1k ohm resistor network\nFarnell no: 137-7053"
- note removed: "Infrared Receiver\n(May optionally replace StartModule)\nVoltage: 2.5-5.5V"
- note removed: "Pull-up resistors for the IR-sensors\n4 x 1k ohm resistor network.\nFarnell no: 923-4519"

Commit message: Routing finished. Playing around with BOM as XSL file.
Parts:
- P4: footprint hrs-fx8c:hrs-fx8c-60p-sv -> hrs-fx8c:hrs-fx8c-60s-sv
Connections:
- net GPIO_MOTOR: now also P4.59 (P59); no longer P4.60 (P60)
- net GPIO_STEERING: now also P4.60 (P60); no longer P4.59 (P59)
- net GPIO_StartModule: now also P4.31 (P31); no longer P4.53 (P53)
- net SC0: now also RN1.4 (R4.1); no longer RN1.3 (R3.1)
- net SC1: now also RN1.2 (R2.1); no longer RN1.1 (R1.1)
- net SC2: now also RN2.4 (R4.1); no longer RN2.3 (R3.1)
- net SC3: now also RN2.2 (R2.1); no longer RN2.1 (R1.1)
- net SC4: now also RN5.8 (R8.1); no longer RN5.7 (R7.1)
- net SC5: now also RN5.6 (R6.1); no longer RN5.5 (R5.1)
- net SC6: now also RN5.4 (R4.1); no longer RN5.3 (R3.1)
- net SC7: now also RN5.2 (R2.1); no longer RN5.1 (R1.1)
- net SD0: now also RN1.3 (R3.1); no longer RN1.4 (R4.1)
- net SD1: now also RN1.1 (R1.1); no longer RN1.2 (R2.1)
- net SD2: now also RN2.3 (R3.1); no longer RN2.4 (R4.1)
- net SD3: now also RN2.1 (R1.1); no longer RN2.2 (R2.1)
- net SD4: now also RN5.7 (R7.1); no longer RN5.8 (R8.1)
- net SD5: now also RN5.5 (R5.1); no longer RN5.6 (R6.1)
- net SD6: now also RN5.3 (R3.1); no longer RN5.4 (R4.1)
- net SD7: now also RN5.1 (R1.1); no longer RN5.2 (R2.1)
Changed lines of the file:
@@
 LIBS:switches
 LIBS:GhostSensorboard-cache
-EELAYER 25 0
+EELAYER 26 0
 EELAYER END
 $Descr A4 11693 8268
 encoding utf-8
 Sheet 1 2
-Title ""
-Date ""
-Rev ""
-Comp ""
+Title "Ghost Sensorboard"
+Date "2017-02-25"
+Rev "1"
+Comp "Frode Lillerud"
 Comment1 ""
 Comment2 ""
@@
 F 0 "P4" H 10200 3950 50  0000 C CNN
 F 1 "CONN_02X30" V 10200 2400 50  0000 C CNN
-F 2 "hrs-fx8c:hrs-fx8c-60p-sv" H 10200 1900 50  0001 C CNN
+F 2 "hrs-fx8c:hrs-fx8c-60s-sv" H 10200 1900 50  0001 C CNN
 F 3 "" H 10200 1900 50  0000 C CNN
 	1    10200 2400
@@
 	1    0    0    -1
 $EndComp
+Text GLabel 850  1350 0    39   Input ~ 0
+SD0
 Text GLabel 850  1450 0    39   Input ~ 0
-SD0
-Text GLabel 850  1350 0    39   Input ~ 0
 SC0
+Text GLabel 850  1150 0    39   Input ~ 0
+SD1
 Text GLabel 850  1250 0    39   Input ~ 0
-SD1
-Text GLabel 850  1150 0    39   Input ~ 0
 SC1
 Wire Wire Line
@@
 Text GLabel 2350 2350 2    39   Input ~ 0
 SC1
+Text GLabel 1800 1350 0    39   Input ~ 0
+SD2
 Text GLabel 1800 1450 0    39   Input ~ 0
-SD2
-Text GLabel 1800 1350 0    39   Input ~ 0
 SC2
+Text GLabel 1800 1150 0    39   Input ~ 0
+SD3
 Text GLabel 1800 1250 0    39   Input ~ 0
-SD3
-Text GLabel 1800 1150 0    39   Input ~ 0
 SC3
 Text GLabel 2350 2850 2    39   Input ~ 0
@@
 Text GLabel 2350 2750 2    39   Input ~ 0
 SC3
+Text GLabel 2850 1550 0    39   Input ~ 0
+SD4
 Text GLabel 2850 1650 0    39   Input ~ 0
-SD4
-Text GLabel 2850 1550 0    39   Input ~ 0
 SC4
+Text GLabel 2850 1350 0    39   Input ~ 0
+SD5
 Text GLabel 2850 1450 0    39   Input ~ 0
-SD5
-Text GLabel 2850 1350 0    39   Input ~ 0
 SC5
+Text GLabel 2850 1150 0    39   Input ~ 0
+SD6
 Text GLabel 2850 1250 0    39   Input ~ 0
-SD6
-Text GLabel 2850 1150 0    39   Input ~ 0
 SC6
+Text GLabel 2850 950  0    39   Input ~ 0
+SD7
 Text GLabel 2850 1050 0    39   Input ~ 0
-SD7
-Text GLabel 2850 950  0    39   Input ~ 0
 SC7
 Wire Wire Line
@@
 Text Notes 5600 6650 2    39   ~ 0
 Level shifting IO signals from 3V3 to 5V.
-Text GLabel 9800 3550 0    39   Input ~ 0
+Text GLabel 9850 2450 0    39   Input ~ 0
 GPIO_StartModule
 Text GLabel 1400 5350 2    39   Input ~ 0
@@
 Text GLabel 9900 950  0    39   Input ~ 0
 GPIO_IR
+Text GLabel 10550 3850 2    39   Input ~ 0
+GPIO_STEERING
 Text GLabel 9850 3850 0    39   Input ~ 0
-GPIO_STEERING
-Text GLabel 10550 3850 2    39   Input ~ 0
 GPIO_MOTOR
 $Comp
@@
 NoConn ~ 10450 1750
 NoConn ~ 10450 2550
-NoConn ~ 9950 2550
 NoConn ~ 9950 3050
 NoConn ~ 9950 3150
@@
 	9950 3450 9800 3450
 Wire Wire Line
-	9800 3550 9950 3550
-Wire Wire Line
 	10600 3450 10450 3450
 Wire Wire Line
@@
 NoConn ~ 10450 3150
 Wire Wire Line
-	10550 3850 10450 3850
-Wire Wire Line
 	10450 3750 10550 3750
 Wire Wire Line
-	9950 3850 9850 3850
-Wire Wire Line
 	9950 950  9900 950
-NoConn ~ 9950 2450
-NoConn ~ 10450 2450
 Wire Wire Line
 	9950 3750 9850 3750
@@
 Wire Wire Line
 	2850 1050 2900 1050
+NoConn ~ 9950 3550
+Wire Wire Line
+	9950 2450 9850 2450
+NoConn ~ 10450 2450
+NoConn ~ 9950 2550
+Wire Wire Line
+	10550 3850 10450 3850
+Wire Wire Line
+	9950 3850 9850 3850
 $EndSCHEMATC

Commit message: Both boards done, and sent to Elecrow.
Connections:
- net GND: no longer P4.36 (P36), P4.38 (P38), P4.40 (P40)
- no-connect marks 23 -> 26
Other:
- note added: "Sharp GP2Y0E02B IR sensors\nI2C address: 0x80\nRange 4-50 cm\nJST SH connectors, 4 pin, 1mm pitch"
- note added: "TCA9548ARGER I2C multiplexer\nI2C address: 0x70"
- note removed: "Sharp GP2Y0E02B IR sensors\nI2C address: 0x??\nRange 4-50 cm\nJST SH connectors, 4 pin, 1mm pitch"
Changed lines of the file:
@@
 	7700 2900 7650 2900
 Text Notes 5950 1900 2    39   ~ 0
-Sharp GP2Y0E02B IR sensors\nI2C address: 0x??\nRange 4-50 cm\nJST SH connectors, 4 pin, 1mm pitch
+Sharp GP2Y0E02B IR sensors\nI2C address: 0x80\nRange 4-50 cm\nJST SH connectors, 4 pin, 1mm pitch
 Text Notes 1000 5800 0    39   ~ 0
 SteeringServo\nPWM signal has been levelshifted from 3V3 to 5V logic.
@@
 	0    -1   -1   0
 $EndComp
-$Comp
-L GND #PWR055
-U 1 1 589AE82D
-P 10750 2650
-F 0 "#PWR055" H 10750 2400 50  0001 C CNN
-F 1 "GND" H 10750 2500 50  0000 C CNN
-F 2 "" H 10750 2650 50  0000 C CNN
-F 3 "" H 10750 2650 50  0000 C CNN
-	1    10750 2650
-	0    -1   -1   0
-$EndComp
-$Comp
-L GND #PWR056
-U 1 1 589AF43D
-P 10750 2750
-F 0 "#PWR056" H 10750 2500 50  0001 C CNN
-F 1 "GND" H 10750 2600 50  0000 C CNN
-F 2 "" H 10750 2750 50  0000 C CNN
-F 3 "" H 10750 2750 50  0000 C CNN
-	1    10750 2750
-	0    -1   -1   0
-$EndComp
-$Comp
-L GND #PWR057
-U 1 1 589AF4DB
-P 10750 2850
-F 0 "#PWR057" H 10750 2600 50  0001 C CNN
-F 1 "GND" H 10750 2700 50  0000 C CNN
-F 2 "" H 10750 2850 50  0000 C CNN
-F 3 "" H 10750 2850 50  0000 C CNN
-	1    10750 2850
-	0    -1   -1   0
-$EndComp
-Wire Wire Line
-	10750 2650 10450 2650
-Wire Wire Line
-	10750 2750 10450 2750
-Wire Wire Line
-	10450 2850 10750 2850
 Wire Wire Line
 	10750 1650 10450 1650
@@
 Wire Wire Line
 	9950 3850 9850 3850
+NoConn ~ 10450 2650
+NoConn ~ 10450 2750
+NoConn ~ 10450 2850
+Text Notes 1350 3950 0    39   ~ 0
+TCA9548ARGER I2C multiplexer\nI2C address: 0x70
 $EndSCHEMATC

Commit message: Startmodule connected to GPIO instead of 3V3 for software power recycle. Motor-pwm connected to IO25 instead of IO34 (which is input only) DRDY connected to IO33 instead of IO35 (which is input only)
Parts:
- Q1, Q2: symbol BSS138 -> BSS138-RESCUE-GhostSensorboard
Connections:
- net +3V3: no longer P1.1 (P1)
- net GPIO_DRDY: now also P4.56 (P56); no longer P4.58 (P58)
- net GPIO_MOTOR: now also P4.53 (P53); no longer P4.59 (P59)
- net GPIO_StartModule_VCC: now reaches P4.32 (P32)
- net GPIO_StartModule_VCC: now also P1.1 (P1)
- no-connect marks 26 -> 25
Other:
- note added: "Startmodule\nUse a female 3pin header.\nAccepts both 3V3 and 5V.\nPower is supplied via GPIO, so that recycle can be done via software."
- note removed: "Startmodule\nUse a female 3pin header.\nAccepts both 3V3 and 5V."
Changed lines of the file:
@@
 EESchema Schematic File Version 2
+LIBS:GhostSensorboard-rescue
 LIBS:power
 LIBS:device
@@
 $EndComp
 $Comp
-L BSS138 Q1
+L BSS138-RESCUE-GhostSensorboard Q1
 U 1 1 5897081C
 P 4150 7400
@@
 $EndComp
 Text Notes 1000 4950 0    39   ~ 0
-Startmodule\nUse a female 3pin header.\nAccepts both 3V3 and 5V.
+Startmodule\nUse a female 3pin header.\nAccepts both 3V3 and 5V.\nPower is supplied via GPIO, so that recycle can be done via software.
 $Comp
 L R_Pack04 RN1
@@
 $EndComp
 Wire Wire Line
-	3300 1350 3400 1350
+	3400 1350 3300 1350
 Wire Wire Line
 	3400 850  3400 1650
@@
 	0    -1   -1   0
 $EndComp
-$Comp
-L +3V3 #PWR028
-U 1 1 589806BE
-P 1400 5150
-F 0 "#PWR028" H 1400 5000 50  0001 C CNN
-F 1 "+3V3" H 1400 5290 50  0000 C CNN
-F 2 "" H 1400 5150 50  0000 C CNN
-F 3 "" H 1400 5150 50  0000 C CNN
-	1    1400 5150
-	0    1    1    0
-$EndComp
 Wire Wire Line
 	1300 5150 1400 5150
@@
 	1300 7050 1450 7050
 $Comp
-L BSS138 Q2
+L BSS138-RESCUE-GhostSensorboard Q2
 U 1 1 58982B38
 P 5900 7400
@@
 Text Notes 6450 4200 0    39   ~ 0
 Gyro/Accelerometer/Compass
-Text GLabel 10550 3750 2    39   Input ~ 0
+Text GLabel 10600 3650 2    39   Input ~ 0
 GPIO_DRDY
 Text GLabel 9850 2750 0    39   Input ~ 0
@@
 Text GLabel 9900 950  0    39   Input ~ 0
 GPIO_IR
-Text GLabel 10550 3850 2    39   Input ~ 0
+Text GLabel 10600 3850 2    39   Input ~ 0
 GPIO_STEERING
-Text GLabel 9850 3850 0    39   Input ~ 0
+Text GLabel 9800 3550 0    39   Input ~ 0
 GPIO_MOTOR
 $Comp
@@
 Wire Wire Line
 	9850 2850 9950 2850
-NoConn ~ 10450 3650
 NoConn ~ 9950 3650
 NoConn ~ 9950 3250
 NoConn ~ 10450 3150
-Wire Wire Line
-	10450 3750 10550 3750
 Wire Wire Line
 	9950 950  9900 950
@@
 Wire Wire Line
 	2850 1050 2900 1050
-NoConn ~ 9950 3550
 Wire Wire Line
 	9950 2450 9850 2450
-NoConn ~ 10450 2450
 NoConn ~ 9950 2550
 Wire Wire Line
-	10550 3850 10450 3850
-Wire Wire Line
-	9950 3850 9850 3850
+	10600 3850 10450 3850
 NoConn ~ 10450 2650
 NoConn ~ 10450 2750
@@
 Text Notes 1350 3950 0    39   ~ 0
 TCA9548ARGER I2C multiplexer\nI2C address: 0x70
+Text GLabel 10500 2450 2    39   Input ~ 0
+GPIO_StartModule_VCC
+Wire Wire Line
+	10450 2450 10500 2450
+Text GLabel 1400 5150 2    39   Input ~ 0
+GPIO_StartModule_VCC
+Wire Wire Line
+	9950 3550 9800 3550
+NoConn ~ 9950 3850
+Wire Wire Line
+	10450 3650 10600 3650
+NoConn ~ 10450 3750
 $EndSCHEMATC
