File: KiCad/GhostSensorboard/Rev2/FreeIMU.sch (KiCad schematic (older format))
At the start: 7 parts, among them U5 MPU-6050, U6 HMC5883

Commit message: Made a connectorboard
Connections:
- net SCL: now also U6.1 (SCL)
- net SDA: now also U6.16 (SDA)
- net MPU_SCL: no longer names the net of U5.7 (AUX_CL)
- net MPU_SCL: no longer U6.1 (SCL)
- net MPU_SDA: no longer names the net of U5.6 (AUX_DA)
- net MPU_SDA: no longer U6.16 (SDA)
- no-connect marks 0 -> 2
Other:
- note removed: "FreeIMU"
Changed lines of the file:
@@
 $Descr A4 11693 8268
 encoding utf-8
-Sheet 2 2
+Sheet 2 3
 Title "Ghost Sensorboard"
 Date "2017-03-10"
@@
 $EndComp
 $Comp
-L GND #PWR074
+L GND #PWR52
 U 1 1 574C3F70
 P 2400 2850
-F 0 "#PWR074" H 2400 2600 50  0001 C CNN
+F 0 "#PWR52" H 2400 2600 50  0001 C CNN
 F 1 "GND" H 2400 2700 50  0000 C CNN
 F 2 "" H 2400 2850 50  0000 C CNN
@@
 FSYNC
 $Comp
-L GND #PWR075
+L GND #PWR53
 U 1 1 574C4065
 P 2700 3850
-F 0 "#PWR075" H 2700 3600 50  0001 C CNN
+F 0 "#PWR53" H 2700 3600 50  0001 C CNN
 F 1 "GND" H 2700 3700 50  0000 C CNN
 F 2 "" H 2700 3850 50  0000 C CNN
@@
 $EndComp
 $Comp
-L GND #PWR076
+L GND #PWR54
 U 1 1 574C40EB
 P 2800 4750
-F 0 "#PWR076" H 2800 4500 50  0001 C CNN
+F 0 "#PWR54" H 2800 4500 50  0001 C CNN
 F 1 "GND" H 2800 4600 50  0000 C CNN
 F 2 "" H 2800 4750 50  0000 C CNN
@@
 $EndComp
 $Comp
-L GND #PWR077
+L GND #PWR55
 U 1 1 574C4E5A
 P 4250 4000
-F 0 "#PWR077" H 4250 3750 50  0001 C CNN
+F 0 "#PWR55" H 4250 3750 50  0001 C CNN
 F 1 "GND" H 4250 3850 50  0000 C CNN
 F 2 "" H 4250 4000 50  0000 C CNN
@@
 	1    0    0    -1
 $EndComp
-Text Notes 2750 1050 0    118  ~ 24
-FreeIMU
 $Comp
 L HMC5883 U6
@@
 	1    0    0    -1
 $EndComp
-Text GLabel 4450 3400 2    60   Input ~ 0
-MPU_SCL
-Text GLabel 4450 3500 2    60   Input ~ 0
-MPU_SDA
-Text GLabel 6450 3450 0    60   Input ~ 0
-MPU_SCL
-Text GLabel 7200 2700 1    60   Input ~ 0
-MPU_SDA
 Text HLabel 6400 3650 0    60   Input ~ 0
 VCC
@@
 $EndComp
 $Comp
-L GND #PWR078
+L GND #PWR56
 U 1 1 574C70FE
 P 9450 4350
-F 0 "#PWR078" H 9450 4100 50  0001 C CNN
+F 0 "#PWR56" H 9450 4100 50  0001 C CNN
 F 1 "GND" H 9450 4200 50  0000 C CNN
 F 2 "" H 9450 4350 50  0000 C CNN
@@
 	4100 3800 4450 3800
 Wire Wire Line
-	4450 3400 4100 3400
-Wire Wire Line
-	4100 3500 4450 3500
-Wire Wire Line
 	4100 3700 4450 3700
 Wire Wire Line
@@
 Text Notes 8550 2800 0    60   ~ 0
 HMC5883 compass\nFarnell no: 197-1743\nI2C address: 0x1E
+NoConn ~ 4100 3400
+NoConn ~ 4100 3500
+Text HLabel 6450 3450 0    60   Input ~ 0
+SCL
+Text HLabel 7200 2700 1    60   Input ~ 0
+SDA
 $EndSCHEMATC
