File: KiCad/GhostSensorboard/Rev2/GhostSensorboard.kicad_pcb (KiCad board)
At the start: 4 copper layers, 60 x 37 mm, 49 parts, among them J2 CONN_02X20, P1 StartModule, P2 SteeringServo, P3 Motor, Q1 BSS138, Q2 BSS138, SW1 SW_Push, U1 TCA9548ARGER, U10 GP2Y0E02B, U11 GP2Y0E02B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

Commit message: Rev2 sent to Elecrow for production
Parts:
- moved C2 6.44 mm to (99.2, 88.9), turned to 180 degrees
- moved RN1 0.97 mm to (114.8, 101.3)
- moved R12 0.83 mm to (110.9, 99.5)
- moved R11 0.82 mm to (107.4, 99.2), turned to 90 degrees
- moved Q1 0.54 mm to (111.3, 105.9)
- moved R14 0.53 mm to (93.8, 110.4)
- moved R5 0.18 mm to (103.3, 81.7), turned to 180 degrees
Connections:
- J2 pad 11: (no net) -> Net-(J2-Pad11)
- J2 pad 12: (no net) -> Net-(J2-Pad12)
- J2 pad 23: (no net) -> IO21
- J2 pad 27: (no net) -> IO16
- J2 pad 28: (no net) -> IO4
- J2 pad 29: (no net) -> Net-(J2-Pad29)
- J2 pad 30: (no net) -> Net-(J2-Pad30)
- J2 pad 31: (no net) -> Net-(J2-Pad31)
- J2 pad 32: (no net) -> Net-(J2-Pad32)
- J2 pad 6: (no net) -> Net-(J2-Pad6)
- RN3 pad 1: SD13 -> SC13
- RN3 pad 2: SC13 -> SD13
- RN3 pad 3: SD12 -> SC12
- RN3 pad 4: SC12 -> SD12
- RN3 pad 5: SD11 -> SC11
- RN3 pad 6: SC11 -> SD11
- RN3 pad 7: SD10 -> SC10
- RN3 pad 8: SC10 -> SD10
Routing:
- net +3V3: track 60.5 -> 308.8 mm, vias 4 -> 6
- net GND: track 14.6 -> 127.8 mm, vias 0 -> 17
- net IO26: track 2.90 -> 39.4 mm, vias 0 -> 3
- net IO27: track 0.00 -> 31.7 mm, vias 0 -> 1
- net SD5: track 0.00 -> 28.1 mm, vias 0 -> 2
- net SC14: track 0.00 -> 27.2 mm, vias 0 -> 2
- net SD14: track 0.00 -> 27.0 mm
- net SD15: track 0.00 -> 27.0 mm, vias 0 -> 2
- net LED: track 0.00 -> 26.0 mm, vias 0 -> 3
- net SC15: track 0.00 -> 25.5 mm, vias 0 -> 2
- net SD3: track 18.1 -> 43.3 mm, vias 0 -> 2
- net SC3: track 16.3 -> 39.7 mm, vias 0 -> 2
- net BUTTON: track 0.00 -> 22.5 mm, vias 0 -> 1
- net IO17: track 29.0 -> 49.4 mm, vias 1 -> 0
- net SC5: track 8.23 -> 26.5 mm, vias 0 -> 2
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- added copper zone on B.Cu, net GND
- added copper zone on F.Cu, net GND
- removed copper zone on 3v3_PLANE, net +3V3
- removed copper zone on GND_PLANE, net GND
Other:
- copper layers 4 -> 2
- board text added: "Encoder"
- board text added: "Ghost Sensorboard, Rev 2 20.mar 2017 Frode Lillerud"
- board text added: "Motor / Start"
- board text added: "Start"
