File: KiCad/GhostSensorboard/Rev2/GhostSensorboard.sch (KiCad schematic (older format))
At the start: 33 parts, among them P1 StartModule, P2 SteeringServo, P3 Motor, P4 CONN_02X30, Q1 BSS138, Q2 BSS138, SW1 SW_Push, U1 TCA9548ARGER, U10 GP2Y0E02B, U11 GP2Y0E02B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

Commit message: Made a connectorboard
Parts:
- removed RN1, RN2: R_Pack04, Resistors_SMD:R_Array_Convex_4x0603, symbol R_Pack04
- removed RN5: R_Pack08, Resistors_SMD:R_Array_Convex_8x0602, symbol R_Pack08
- removed U1: TCA9548ARGER, Housings_DFN_QFN:QFN-24_4x4mm_Pitch0.5mm, symbol TCA9548ARGER
- removed U10, U11, U12, U2, U3, U7, U8, U9: GP2Y0E02B, Connectors_JST:JST_SH_BM04B-SRSS-TB_04x1.00mm_Straight, symbol GP2Y0E02B
- added J1: CONN_02X08, Pin_Headers:Pin_Header_Straight_2x08_Pitch2.54mm, symbol CONN_02X08
- added R11: 2k2, Resistors_SMD:R_0603, symbol R
- R1, R10, R2, R3, R4, R5, R6, R7, R8, R9: footprint Resistors_SMD:R_0603_HandSoldering -> Resistors_SMD:R_0603
Connections:
- net +3V3: now also J1.1 (P1), J1.3 (P3), R11.1
- net +5V: now also J1.13 (P13), J1.15 (P15)
- net GND: now also J1.14 (P14), J1.16 (P16), J1.2 (P2), J1.4 (P4)
- net GPIO_SCL_0: now reaches R1.2
- net GPIO_SCL_0: now also P4.51 (P51)
- net GPIO_SCL renamed GPIO_SCL_1
- net GPIO_SCL_1: no longer P4.51 (P51)
- net GPIO_SDA renamed GPIO_SDA_0
- net GPIO_SDA_0: now also R11.2; no longer R10.2
- new net GPIO_16: J1.7 (P7)
- new net GPIO_17: J1.9 (P9)
- new net GPIO_18: J1.11 (P11)
- new net GPIO_19: J1.12 (P12)
- new net GPIO_21: J1.10 (P10)
- new net GPIO_32: J1.6 (P6)
- new net GPIO_33: J1.8 (P8)
- new net GPIO_4: J1.5 (P5)
- new net GPIO_SDA_1: R10.2
Other:
- note added: "TODO!!! DOUBLECHECK ALL THE PINS!!\n"
- note removed: "Pull-up resistors for the IR-sensors\n4 x 1k ohm resistor network.\nFarnell no: 923-4519\n8 x 1k ohm resistor network\nFarnell no: 137-7053"
- note removed: "Sharp GP2Y0E02B IR sensors\nI2C address: 0x80\nRange 4-50 cm\nJST SH connectors, 4 pin, 1mm pitch"
- note removed: "TCA9548ARGER I2C multiplexer\nI2C address: 0x70"
- moved on the sheet: C1, C2, D1, Q1, Q2, R10, R2, R3, R4, R5, R6, R7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

Commit message: Working on the Encoder
Parts:
- removed J1: CONN_02X08, Pin_Headers:Pin_Header_Straight_2x08_Pitch2.54mm, symbol CONN_02X08
- added J1: CONN_02X05, Pin_Headers:Pin_Header_Straight_2x05_Pitch2.54mm, symbol CONN_02X05
Connections:
- net +BATT is gone; now on net +5V: P3.2 (P2)
- net +3V3: now also J1.1 (P1)
- net +5V: now also J1.2 (P2)
- net GND: now also J1.10 (P10)
- net GPIO_16: now also J1.5 (P5)
- net GPIO_17: now also J1.7 (P7)
- net GPIO_18: now also J1.9 (P9)
- net GPIO_21: now also J1.8 (P8)
- net GPIO_32: now also J1.4 (P4)
- net GPIO_33: now also J1.6 (P6)
- net GPIO_4: now also J1.3 (P3)
- no-connect marks 25 -> 26
Other:
- note removed: "Gyro/Accelerometer/Compass"

Commit message: Ready to start routing. Schematics should be done.
Parts:
- removed J1: CONN_02X05, Pin_Headers:Pin_Header_Straight_2x05_Pitch2.54mm, symbol CONN_02X05
- removed P4: CONN_02X30, hrs-fx8c:hrs-fx8c-60s-sv, symbol CONN_02X30
- added J2: CONN_02X20, hrs-fx8c:hrs-fx8c-40s-sv5, symbol CONN_02X20
- added R14: 270, Resistors_SMD:R_0402, symbol R
- added R15: 10k, Resistors_SMD:R_0402, symbol R
- added U5: Transmissive_Photo_Interrupter, Pin_Headers:Pin_Header_Straight_1x04_Pitch2.54mm, symbol Transmissive_Photo_Interrupter
- R1, R10, R11, R2, R3, R4, R5, R6, R7, R8, R9: footprint Resistors_SMD:R_0603 -> Resistors_SMD:R_0402
Connections:
- net GPIO_LED is gone; now on net +3V3: R5.2
- net +3V3: now also J2.10 (P10), J2.7 (P7), J2.8 (P8), J2.9 (P9)
- net +5V: now also J2.35 (P35), J2.36 (P36), J2.37 (P37), J2.38 (P38), J2.39 (P39), J2.40 (P40), R14.2, R15.1
- net GND: now also J2.13 (P13), J2.14 (P14), J2.15 (P15), J2.16 (P16), J2.17 (P17), J2.18 (P18), J2.19 (P19), J2.20 (P20), U5.2 (CATHODE), U5.4 (EMITTER); no longer D1.1 (K)
- net GPIO_BUTTON renamed BUTTON
- net BUTTON: now also J2.25 (P25)
- net GPIO_IR renamed IO22
- net IO22: now also J2.22 (P22)
- net GPIO_MOTOR renamed IO27
- net IO27: now also J2.1 (P1)
- net GPIO_SCL_0 renamed IO14
- net IO14: now also J2.34 (P34)
- net GPIO_SCL_1 renamed IO32
- net IO32: now also J2.5 (P5)
- net GPIO_SDA_0 renamed IO13
- net IO13: now also J2.33 (P33)
- net GPIO_SDA_1 renamed IO33
- net IO33: now also J2.4 (P4)
- net GPIO_STEERING renamed IO26
- net IO26: now also J2.2 (P2)
- net GPIO_StartModule renamed IO25
- net IO25: now also J2.3 (P3)
- net GPIO_StartModule_VCC renamed IO17
- net IO17: now also J2.26 (P26)
- net MotorPWM renamed MOTOR_5V_PWM
- net SteeringPWM renamed STEERING_5V_PWM
- new net: R14.1, U5.1 (ANODE)
- new net ENCODER: J2.24 (P24), R15.2, U5.3 (COLLECTOR)
- new net IO16: J2.27 (P27)
- new net IO21: J2.23 (P23)
- new net IO4: J2.28 (P28)
- new net LED: D1.1 (K), J2.21 (P21)
- no-connect marks 26 -> 11
Other:
- note added: "A shield for the Ghost32 board.\nContains sensors and connectors."
- note added: "Bottom connector, 40 pin\nHirose FX8C-40S-SV5\nFarnell no: 249-8688"
- note added: "Encoder\nKTIR0611S"
- note added: "Mapping of ESP32 GPIO's \nto physical devices"
- note added: "NB, IO23 is dedicated to LED\nNB, IO32 (SCL) and IO33 (SDA) is dedicated to I2C"
- note added: "Pull-up resistors for \nI2C channel 0"
- note added: "Pull-up resistors for \nI2C channel 1"
- note removed: "A shield for the Ghost32 board.\nContains all the sensors and connectors."
- note removed: "Pull-up resistors for I2C"
- note removed: "TODO!!! DOUBLECHECK ALL THE PINS!!\n"
- moved on the sheet: C1, C2, D1, R1, R10, R11, R2, R4, R5, R9, SW1, U4

Commit message: Rev2 sent to Elecrow for production
Other:
- moved on the sheet: P1, P2, P3
