File: KiCad/GhostESP32/Rev3/GhostESP32.sch (KiCad schematic (older format))
At the start: 38 parts, among them J1 CONN_02X05, J2 USB_OTG, J3 CONN_01X14, J4 CONN_01X10, Q1 Q_NPN_BEC, Q2 Q_NPN_BEC, Q3 Q_NPN_BEC, SW1 SW_SPDT, U1 MPU-9250, U2 NCP1117ST33T3G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

Commit message: Working on Rev3 of GhostESP32
Parts:
- removed C9: 1nF, Capacitors_SMD:C_0402, symbol C
- removed R10: 470, Resistors_SMD:R_0402, symbol R
- added D3, D4, D6: ESD, Diodes_SMD:D_0603, symbol D_Zener_Small_ALT
- added R5, R6: 68, Resistors_SMD:R_0402, symbol R
- added U5: TMP102, NorBotKiCadFootprints:SOT563, symbol TMP102
- C10: value 1nF -> 1uF
- D5: footprint Diodes_SMD:D_SMA_Standard -> Diodes_SMD:D_SMA
Connections:
- net +3V3: now also J3.3 (P3), U5.5 (V+); no longer J3.1 (P1)
- net +BATT: now also C1.1, D5.1 (K), J3.1 (P1), R1.1, U2.3 (VI); no longer J3.13 (P13)
- net EN: now also J3.14 (P14), SW1.3 (C); no longer J4.7 (P7)
- net GND: now also J3.2 (P2), D3.2 (A), D4.2 (A), D6.2 (A), U5.2 (GND), U5.4 (ADD0); no longer J3.14 (P14)
- net I34: now also J3.11 (P11); no longer J4.3 (P3)
- net I36: now also J3.13 (P13); no longer J4.8 (P8)
- net I39: now also J3.12 (P12), U5.3 (ALERT); no longer J4.9 (P9)
- net IO14: now also J3.9 (P9); no longer J4.6 (P6)
- net IO16: now also J4.4 (P4); no longer J3.9 (P9)
- net IO17: now also J4.5 (P5); no longer J4.4 (P4)
- net IO18: now also J4.6 (P6); no longer J3.8 (P8)
- net IO19: now also J4.7 (P7); no longer J3.12 (P12)
- net IO21: now also J4.8 (P8); no longer J3.7 (P7)
- net IO22: now also J4.9 (P9); no longer J3.11 (P11)
- net IO23: now also R12.1; no longer R12.2
- net IO25: now also J3.6 (P6); no longer J3.3 (P3)
- net IO26: now also J3.5 (P5); no longer J4.2 (P2)
- net IO27: now also J3.4 (P4); no longer J3.2 (P2)
- net IO32/SCL: now also J3.8 (P8), R8.2, U4.8 (IO32), U5.1 (SCL); no longer J3.4 (P4)
- net IO33/SDA: now also J3.7 (P7), R9.2, U4.9 (IO33), U5.6 (SDA); no longer J3.5 (P5)
- net IO4: now also J4.3 (P3); no longer J4.5 (P5)
- net LED: now also J4.2 (P2); no longer J3.6 (P6)
- net USB_DN: now also R6.1; no longer J2.2 (D-)
- net USB_DP: now also R5.1; no longer J2.3 (D+)
- net VBUS: now reaches D5.2 (A), J2.1 (VBUS)
- net VBUS: now also C7.1, C8.1, J4.1 (P1), U3.8 (VBUS), D3.1 (K)
- net at Q3.1 (B): now also R12.2; no longer R12.1
- removed net +5V: C1.1, C7.1, C8.1, D5.1 (K), J4.1 (P1), R1.1, U2.3 (VI), U3.8 (VBUS)
- removed net IO32: R9.2, U4.8 (IO32)
- removed net IO33: R8.2, U4.9 (IO33)
- new net: D6.1 (K), J2.2 (D-), R6.2
- new net: D4.1 (K), J2.3 (D+), R5.2
Other:
- note added: "Batt (3.5V - 20V)"
- note added: "ESD suppressors\nFarnell no: 238-3318"
- note added: "I2C pull-ups"
- note added: "TMP102 temperature\nI2C address: 0x48\nFarnell no: 165-2477"
- note removed: "I2C pull-ups, not-connected.\nOnly used when using \nboard in single-board mode."
- moved on the sheet: C10, C11, C12, C13, C4, C6, D2, J1, J2, Q3, R11, R12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
