File: KiCad/GhostSensorboard/Rev3/GhostSensorboard.kicad_pcb (KiCad board)
At the start: 2 copper layers, 60 x 37 mm, 60 parts, among them J1 CONN_01X14, J2 CONN_01X10, P1 StartModule, P2 SteeringServo, P3 Motor, Q1 BSS138, Q2 BSS138, SW1 SW_Push, U1 TCA9548ARGER, U10 GP2Y0E02B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

Commit message: Update to rev 3
Parts:
- removed the REF** at (163.3, 81.6)
- removed RN1, RN2, RN3, RN4: R_Pack08, Resistors_SMD:R_Array_Convex_8x0602
- removed U15, U16, U17, U18, U19, U20, U21: GP2Y0E02B, Connectors_JST:JST_SH_BM04B-SRSS-TB_04x1.00mm_Straight
- added C4: 0.1uF, Capacitors_SMD:C_0402, F.Cu at (121.6, 110.9)
- added R19: 1k, Resistors_SMD:R_0402, F.Cu at (117.1, 94.3)
- added R20: 1k, Resistors_SMD:R_0402, F.Cu at (122.3, 84.4)
- added R21: 1k, Resistors_SMD:R_0402, F.Cu at (123.9, 84.4)
- added R22: 1k, Resistors_SMD:R_0402, F.Cu at (117.2, 84.9)
- added R23: 1k, Resistors_SMD:R_0402, F.Cu at (117.2, 87.2)
- added R24: 1k, Resistors_SMD:R_0402, F.Cu at (132.6, 93.0)
- added R25: 1k, Resistors_SMD:R_0402, F.Cu at (133.9, 92.9)
- added R26: 1k, Resistors_SMD:R_0402, F.Cu at (121.9, 92.9)
- added R27: 1k, Resistors_SMD:R_0402, F.Cu at (123.8, 93.0)
- added R28: 1k, Resistors_SMD:R_0402, F.Cu at (131.7, 84.8)
- added R29: 1k, Resistors_SMD:R_0402, F.Cu at (133.3, 84.8)
- added R30: 1k, Resistors_SMD:R_0402, F.Cu at (122.8, 101.4)
- added R31: 1k, Resistors_SMD:R_0402, F.Cu at (124.2, 101.3)
- added REF**: MountingHole_3.2mm_M3_Pad_Via, Mounting_Holes:MountingHole_3.2mm_M3_Pad_Via, F.Cu at (111.2, 110.5)
- added REF**: MountingHole_3.2mm_M3_Pad_Via, Mounting_Holes:MountingHole_3.2mm_M3_Pad_Via, F.Cu at (111.2, 81.5)
- added REF**: MountingHole_3.2mm_M3_Pad_Via, Mounting_Holes:MountingHole_3.2mm_M3_Pad_Via, F.Cu at (163.2, 110.5)
- added REF**: MountingHole_3.2mm_M3_Pad_Via, Mounting_Holes:MountingHole_3.2mm_M3_Pad_Via, F.Cu at (163.2, 81.5)
- added SW2: SW_SPDT, NorBotKiCadFootprints:MFP106D, F.Cu at (151.7, 105.4)
- C1: value 0.1uF -> 1uF
- R10, R13, R9: value 2k2 -> 1k
- R2: value 100 -> 33-1k ohm
- U14: value GP2Y0E02B -> MIC5219-5.0; footprint Connectors_JST:JST_SH_BM04B-SRSS-TB_04x1.00mm_Straight -> TO_SOT_Packages_SMD:SOT-23-5
- U4: value TSOP753 -> TSOP752-TSOP754
- U6: value MIC5219-5.0BM5 -> NeoPixelNano; footprint TO_SOT_Packages_SMD:SOT-23-5 -> NorBotKiCadFootprints:NeoPixelNano
- U9: value TCA9548ARGER -> NeoPixelNano; footprint Housings_DFN_QFN:QFN-24_4x4mm_Pitch0.5mm_NoMask -> NorBotKiCadFootprints:NeoPixelNano
- moved R9 104.2 mm to (116.9, 100.2), turned to 90 degrees
- moved U6 94.8 mm to (118.1, 111.0), turned to 90 degrees
- moved D4 91.5 mm to (133.5, 106.0), turned to 90 degrees
- moved R13 85.8 mm to (117.1, 92.2), turned to 90 degrees
- moved U9 79.8 mm to (118.1, 79.9), turned to 180 degrees
- moved R10 79.4 mm to (116.9, 102.2), turned to 270 degrees
- moved U4 77.0 mm to (139.6, 105.2), turned to 90 degrees
- moved R16 71.5 mm to (128.3, 103.4), turned to 90 degrees
- moved D2 70.0 mm to (128.4, 106.1), turned to 90 degrees
- moved D1 68.6 mm to (136.3, 106.2), turned to 90 degrees
- moved R12 65.5 mm to (141.3, 91.1), turned to 90 degrees
- moved R2 64.6 mm to (143.4, 106.1), turned to 270 degrees
- moved R1 63.7 mm to (141.2, 84.3), turned to 90 degrees
- moved R5 63.4 mm to (136.4, 103.3), turned to 90 degrees
- moved Q2 61.9 mm to (153.9, 91.3)
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Connections:
- BT1 pad 1: (no net) -> Net-(BT1-Pad1)
- J1 pad 10: IO13 -> (no net)
- J1 pad 7: (no net) -> IO33/SDA
- J1 pad 9: IO14 -> (no net)
- J2 pad 4: (no net) -> IO16
- R1 pad 2: IO14 -> IO32/SCL
- R10 pad 2: IO33/SCL -> SC0
- R11 pad 2: IO13 -> IO33/SDA
- R13 pad 2: Net-(R13-Pad2) -> SD1
- R9 pad 2: IO32/SCL -> SD0
- U1 pad 19: IO14 -> IO32/SCL
- U1 pad 20: IO13 -> IO33/SDA
- U14 pad 1: SC8 -> +BATT
- U14 pad 2: SD8 -> GND
- U14 pad 3: GND -> ENABLE5V
- U14 pad 4: +3V3 -> (no net)
- U6 pad 1: +BATT -> Net-(U6-Pad1)
- U6 pad 3: ENABLE5V -> IO16
- U6 pad 4: (no net) -> +5V
- U9 pad 1: SD8 -> (no net)
- U9 pad 2: SC8 -> GND
- U9 pad 3: SD9 -> Net-(U6-Pad1)
- U9 pad 4: SC9 -> +5V
Routing:
- net GND: track 0.00 -> 273.1 mm, vias 0 -> 17
- net +3V3: track 0.00 -> 204.2 mm, vias 0 -> 14
- net +5V: track 0.00 -> 123.6 mm, vias 0 -> 4
- net +BATT: track 0.00 -> 74.2 mm, vias 0 -> 1
- net SD3: track 0.00 -> 50.6 mm, vias 0 -> 4
- net ENCODER: track 0.00 -> 50.6 mm
- net IO26: track 0.00 -> 47.0 mm, vias 0 -> 2
- net SC3: track 0.00 -> 43.5 mm, vias 0 -> 4
- net SC0: track 0.00 -> 42.6 mm, vias 0 -> 2
- net SD0: track 0.00 -> 41.4 mm, vias 0 -> 2
- net SD1: track 0.00 -> 41.1 mm, vias 0 -> 4
- net IO25: track 0.00 -> 39.4 mm
- net SC5: track 0.00 -> 38.5 mm, vias 0 -> 4
- net SD7: track 0.00 -> 38.4 mm
- net SC7: track 0.00 -> 37.4 mm
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Other:
- board text added: "Ghost Sensorboard, Rev 3 21.07.2017 Frode Lillerud"
