File: KiCad/GhostSensorboard/Rev3/GhostSensorboard.sch (KiCad schematic (older format))
At the start: 37 parts, among them J1 CONN_01X14, J2 CONN_01X10, P1 StartModule, P2 SteeringServo, P3 Motor, Q1 BSS138, Q2 BSS138, SW1 SW_Push, SW2 SW_SPDT, U5 Transmissive_Photo_Interrupter

Commit message: Update to rev 3
Parts:
- C4: renamed from C?; footprint (none) -> Capacitors_SMD:C_0402
- SW2: footprint (none) -> NorBotKiCadFootprints:MFP106D
- U4: renamed from U?; footprint (none) -> NorBotKiCadFootprints:TSOP75x
- U6, U9: renamed from U?; footprint (none) -> NorBotKiCadFootprints:NeoPixelNano
- gave numbers to parts that had none: 1
Connections:
- net IO33/SCL is gone; now on net IO33/SDA: R11.2
- no-connect marks 6 -> 10

Commit message: A massive bunch of former changes waiting to be committed.
Parts:
- BT1: symbol Battery_Cell -> GhostSensorboard-rescue:Battery_Cell-RESCUE-GhostSensorboard
- C1, C2: symbol C -> GhostSensorboard-rescue:C-RESCUE-GhostSensorboard
- C3, C4: symbol C_Small -> GhostSensorboard-rescue:C_Small-RESCUE-GhostSensorboard
- D1, D2, D3, D4: symbol LED -> GhostSensorboard-rescue:LED-RESCUE-GhostSensorboard
- J1: symbol CONN_01X14 -> GhostSensorboard-rescue:CONN_01X14-RESCUE-GhostSensorboard
- J2: symbol CONN_01X10 -> GhostSensorboard-rescue:CONN_01X10-RESCUE-GhostSensorboard
- P1, P2, P3: symbol CONN_01X03 -> GhostSensorboard-rescue:CONN_01X03-RESCUE-GhostSensorboard
- Q1, Q2: symbol BSS138-RESCUE-GhostSensorboard -> GhostSensorboard-rescue:BSS138-RESCUE-GhostSensorboard
- R1, R11, R14, R15, R16, R17, R18, R2, R3, R4, R5, R6, R7, R8: symbol R -> GhostSensorboard-rescue:R-RESCUE-GhostSensorboard
- SW1: symbol SW_Push -> GhostSensorboard-rescue:SW_Push-RESCUE-GhostSensorboard
- SW2: symbol SW_SPDT -> GhostSensorboard-rescue:SW_SPDT-RESCUE-GhostSensorboard
- U14: symbol MIC5219-5.0 -> GhostSensorboard-rescue:MIC5219-5.0-RESCUE-GhostSensorboard
- U4: symbol TSOP752-TSOP754 -> NorBot:TSOP752-TSOP754
- U5: symbol Transmissive_Photo_Interrupter -> NorBot:Transmissive_Photo_Interrupter
- U6, U9: symbol NeoPixelNano -> NorBot:NeoPixelNano
