File: KiCad/GhostSensorboard/Rev3/IRSensors.sch (KiCad schematic (older format))
At the start: 26 parts, among them U1 TCA9548ARGER, U10 GP2Y0E02B, U11 GP2Y0E02B, U12 GP2Y0E02B, U13 GP2Y0E02B, U2 GP2Y0E02B, U3 GP2Y0E02B, U7 GP2Y0E02B, U8 GP2Y0E02B

Commit message: Update to rev 3
Parts:
- R10, R13, R19, R20, R21, R22, R23, R24, R25, R26, R27, R28, R29, R30, R31, R9: renamed from R?; footprint (none) -> Resistors_SMD:R_0402
Changed lines of the file:
@@
 $EndComp
 $Comp
-L GND #PWR38
+L GND #PWR043
 U 1 1 58C891DA
 P 4100 4000
-F 0 "#PWR38" H 4100 3750 50  0001 C CNN
+F 0 "#PWR043" H 4100 3750 50  0001 C CNN
 F 1 "GND" H 4105 3827 50  0000 C CNN
 F 2 "" H 4100 4000 50  0001 C CNN
@@
 	3850 2250 4200 2250
 $Comp
-L +3V3 #PWR35
+L +3V3 #PWR044
 U 1 1 58C89F76
 P 3850 2100
-F 0 "#PWR35" H 3850 1950 50  0001 C CNN
+F 0 "#PWR044" H 3850 1950 50  0001 C CNN
 F 1 "+3V3" H 3865 2273 50  0000 C CNN
 F 2 "" H 3850 2100 50  0001 C CNN
@@
 	9150 4400 9300 4400
 $Comp
-L GND #PWR48
+L GND #PWR045
 U 1 1 58C9A570
 P 8350 2150
-F 0 "#PWR48" H 8350 1900 50  0001 C CNN
+F 0 "#PWR045" H 8350 1900 50  0001 C CNN
 F 1 "GND" V 8355 2022 50  0000 R CNN
 F 2 "" H 8350 2150 50  0001 C CNN
@@
 $EndComp
 $Comp
-L GND #PWR49
+L GND #PWR046
 U 1 1 58C9ABDE
 P 8350 2900
-F 0 "#PWR49" H 8350 2650 50  0001 C CNN
+F 0 "#PWR046" H 8350 2650 50  0001 C CNN
 F 1 "GND" V 8355 2772 50  0000 R CNN
 F 2 "" H 8350 2900 50  0001 C CNN
@@
 $EndComp
 $Comp
-L GND #PWR50
+L GND #PWR047
 U 1 1 58C9AC15
 P 8350 3650
-F 0 "#PWR50" H 8350 3400 50  0001 C CNN
+F 0 "#PWR047" H 8350 3400 50  0001 C CNN
 F 1 "GND" V 8355 3522 50  0000 R CNN
 F 2 "" H 8350 3650 50  0001 C CNN
@@
 $EndComp
 $Comp
-L GND #PWR51
+L GND #PWR048
 U 1 1 58C9AF22
 P 8350 4400
-F 0 "#PWR51" H 8350 4150 50  0001 C CNN
+F 0 "#PWR048" H 8350 4150 50  0001 C CNN
 F 1 "GND" V 8355 4272 50  0000 R CNN
 F 2 "" H 8350 4400 50  0001 C CNN
@@
 $EndComp
 $Comp
-L GND #PWR56
+L GND #PWR049
 U 1 1 58C9B715
 P 10250 2150
-F 0 "#PWR56" H 10250 1900 50  0001 C CNN
+F 0 "#PWR049" H 10250 1900 50  0001 C CNN
 F 1 "GND" V 10255 2022 50  0000 R CNN
 F 2 "" H 10250 2150 50  0001 C CNN
@@
 $EndComp
 $Comp
-L GND #PWR57
+L GND #PWR050
 U 1 1 58C9B74C
 P 10250 2900
-F 0 "#PWR57" H 10250 2650 50  0001 C CNN
+F 0 "#PWR050" H 10250 2650 50  0001 C CNN
 F 1 "GND" V 10255 2772 50  0000 R CNN
 F 2 "" H 10250 2900 50  0001 C CNN
@@
 $EndComp
 $Comp
-L GND #PWR58
+L GND #PWR051
 U 1 1 58C9B783
 P 10250 3650
-F 0 "#PWR58" H 10250 3400 50  0001 C CNN
+F 0 "#PWR051" H 10250 3400 50  0001 C CNN
 F 1 "GND" V 10255 3522 50  0000 R CNN
 F 2 "" H 10250 3650 50  0001 C CNN
@@
 $EndComp
 $Comp
-L GND #PWR59
+L GND #PWR052
 U 1 1 58C9B7BA
 P 10250 4400
-F 0 "#PWR59" H 10250 4150 50  0001 C CNN
+F 0 "#PWR052" H 10250 4150 50  0001 C CNN
 F 1 "GND" V 10255 4272 50  0000 R CNN
 F 2 "" H 10250 4400 50  0001 C CNN
@@
 	8250 4400 8350 4400
 $Comp
-L +3V3 #PWR41
+L +3V3 #PWR053
 U 1 1 58C9DB9B
 P 7250 1850
-F 0 "#PWR41" H 7250 1700 50  0001 C CNN
+F 0 "#PWR053" H 7250 1700 50  0001 C CNN
 F 1 "+3V3" V 7265 1978 50  0000 L CNN
 F 2 "" H 7250 1850 50  0001 C CNN
@@
 $EndComp
 $Comp
-L +3V3 #PWR42
+L +3V3 #PWR054
 U 1 1 58C9E117
 P 7250 2600
-F 0 "#PWR42" H 7250 2450 50  0001 C CNN
+F 0 "#PWR054" H 7250 2450 50  0001 C CNN
 F 1 "+3V3" V 7265 2728 50  0000 L CNN
 F 2 "" H 7250 2600 50  0001 C CNN
@@
 $EndComp
 $Comp
-L +3V3 #PWR43
+L +3V3 #PWR055
 U 1 1 58C9E14E
 P 7250 3350
-F 0 "#PWR43" H 7250 3200 50  0001 C CNN
+F 0 "#PWR055" H 7250 3200 50  0001 C CNN
 F 1 "+3V3" V 7265 3478 50  0000 L CNN
 F 2 "" H 7250 3350 50  0001 C CNN
@@
 $EndComp
 $Comp
-L +3V3 #PWR44
+L +3V3 #PWR056
 U 1 1 58C9E185
 P 7250 4100
-F 0 "#PWR44" H 7250 3950 50  0001 C CNN
+F 0 "#PWR056" H 7250 3950 50  0001 C CNN
 F 1 "+3V3" V 7265 4228 50  0000 L CNN
 F 2 "" H 7250 4100 50  0001 C CNN
@@
 $EndComp
 $Comp
-L +3V3 #PWR52
+L +3V3 #PWR057
 U 1 1 58C9FCAA
 P 9100 1850
-F 0 "#PWR52" H 9100 1700 50  0001 C CNN
+F 0 "#PWR057" H 9100 1700 50  0001 C CNN
 F 1 "+3V3" V 9115 1978 50  0000 L CNN
 F 2 "" H 9100 1850 50  0001 C CNN
@@
 $EndComp
 $Comp
-L +3V3 #PWR53
+L +3V3 #PWR058
 U 1 1 58C9FCE1
 P 9100 2600
-F 0 "#PWR53" H 9100 2450 50  0001 C CNN
+F 0 "#PWR058" H 9100 2450 50  0001 C CNN
 F 1 "+3V3" V 9115 2728 50  0000 L CNN
 F 2 "" H 9100 2600 50  0001 C CNN
@@
 $EndComp
 $Comp
-L +3V3 #PWR54
+L +3V3 #PWR059
 U 1 1 58C9FD18
 P 9100 3350
-F 0 "#PWR54" H 9100 3200 50  0001 C CNN
+F 0 "#PWR059" H 9100 3200 50  0001 C CNN
 F 1 "+3V3" V 9115 3478 50  0000 L CNN
 F 2 "" H 9100 3350 50  0001 C CNN
@@
 $EndComp
 $Comp
-L +3V3 #PWR55
+L +3V3 #PWR060
 U 1 1 58C9FD4F
 P 9100 4100
-F 0 "#PWR55" H 9100 3950 50  0001 C CNN
+F 0 "#PWR060" H 9100 3950 50  0001 C CNN
 F 1 "+3V3" V 9115 4228 50  0000 L CNN
 F 2 "" H 9100 4100 50  0001 C CNN
@@
 	1150 3700 1400 3700
 $Comp
-L +3V3 #PWR36
+L +3V3 #PWR061
 U 1 1 58CA550D
 P 1900 2100
-F 0 "#PWR36" H 1900 1950 50  0001 C CNN
+F 0 "#PWR061" H 1900 1950 50  0001 C CNN
 F 1 "+3V3" H 1915 2273 50  0000 C CNN
 F 2 "" H 1900 2100 50  0001 C CNN
@@
 TCA9548ARGER I2C multiplexer\nI2C address: 0x70\nFarnell no: 269-0239
 $Comp
-L R_Small R?
+L R_Small R23
 U 1 1 5945CFBC
 P 1500 2900
-F 0 "R?" V 1550 3050 50  0000 C CNN
+F 0 "R23" V 1550 3050 50  0000 C CNN
 F 1 "1k" V 1500 2900 50  0000 C CNN
-F 2 "" H 1500 2900 50  0001 C CNN
+F 2 "Resistors_SMD:R_0402" H 1500 2900 50  0001 C CNN
 F 3 "" H 1500 2900 50  0001 C CNN
 	1    1500 2900
@@
 $EndComp
 $Comp
-L R_Small R?
+L R_Small R22
 U 1 1 5945F8C2
 P 1500 2800
-F 0 "R?" V 1550 2950 50  0000 C CNN
+F 0 "R22" V 1550 2950 50  0000 C CNN
 F 1 "1k" V 1500 2800 50  0000 C CNN
-F 2 "" H 1500 2800 50  0001 C CNN
+F 2 "Resistors_SMD:R_0402" H 1500 2800 50  0001 C CNN
 F 3 "" H 1500 2800 50  0001 C CNN
 	1    1500 2800
@@
 $EndComp
 $Comp
-L R_Small R?
+L R_Small R21
 U 1 1 5945F8EE
 P 1500 2700
-F 0 "R?" V 1550 2850 50  0000 C CNN
+F 0 "R21" V 1550 2850 50  0000 C CNN
 F 1 "1k" V 1500 2700 50  0000 C CNN
-F 2 "" H 1500 2700 50  0001 C CNN
+F 2 "Resistors_SMD:R_0402" H 1500 2700 50  0001 C CNN
 F 3 "" H 1500 2700 50  0001 C CNN
 	1    1500 2700
@@
 $EndComp
 $Comp
-L R_Small R?
+L R_Small R20
 U 1 1 5945F91C
 P 1500 2600
-F 0 "R?" V 1550 2750 50  0000 C CNN
+F 0 "R20" V 1550 2750 50  0000 C CNN
 F 1 "1k" V 1500 2600 50  0000 C CNN
-F 2 "" H 1500 2600 50  0001 C CNN
+F 2 "Resistors_SMD:R_0402" H 1500 2600 50  0001 C CNN
 F 3 "" H 1500 2600 50  0001 C CNN
 	1    1500 2600
@@
 $EndComp
 $Comp
-L R_Small R?
+L R_Small R19
 U 1 1 5945F950
 P 1500 2500
-F 0 "R?" V 1550 2650 50  0000 C CNN
+F 0 "R19" V 1550 2650 50  0000 C CNN
 F 1 "1k" V 1500 2500 50  0000 C CNN
-F 2 "" H 1500 2500 50  0001 C CNN
+F 2 "Resistors_SMD:R_0402" H 1500 2500 50  0001 C CNN
 F 3 "" H 1500 2500 50  0001 C CNN
 	1    1500 2500
@@
 $EndComp
 $Comp
-L R_Small R?
+L R_Small R13
 U 1 1 5945F986
 P 1500 2400
-F 0 "R?" V 1550 2550 50  0000 C CNN
+F 0 "R13" V 1550 2550 50  0000 C CNN
 F 1 "1k" V 1500 2400 50  0000 C CNN
-F 2 "" H 1500 2400 50  0001 C CNN
+F 2 "Resistors_SMD:R_0402" H 1500 2400 50  0001 C CNN
 F 3 "" H 1500 2400 50  0001 C CNN
 	1    1500 2400
@@
 $EndComp
 $Comp
-L R_Small R?
+L R_Small R10
 U 1 1 5945F9C4
 P 1500 2300
-F 0 "R?" V 1550 2450 50  0000 C CNN
+F 0 "R10" V 1550 2450 50  0000 C CNN
 F 1 "1k" V 1500 2300 50  0000 C CNN
-F 2 "" H 1500 2300 50  0001 C CNN
+F 2 "Resistors_SMD:R_0402" H 1500 2300 50  0001 C CNN
 F 3 "" H 1500 2300 50  0001 C CNN
 	1    1500 2300
@@
 $EndComp
 $Comp
-L R_Small R?
+L R_Small R9
 U 1 1 5945F9FA
 P 1500 2200
-F 0 "R?" V 1550 2350 50  0000 C CNN
+F 0 "R9" V 1550 2350 50  0000 C CNN
 F 1 "1k" V 1500 2200 50  0000 C CNN
-F 2 "" H 1500 2200 50  0001 C CNN
+F 2 "Resistors_SMD:R_0402" H 1500 2200 50  0001 C CNN
 F 3 "" H 1500 2200 50  0001 C CNN
 	1    1500 2200
@@
 $EndComp
 $Comp
-L R_Small R?
+L R_Small R31
 U 1 1 59461171
 P 1500 3700
-F 0 "R?" V 1550 3850 50  0000 C CNN
+F 0 "R31" V 1550 3850 50  0000 C CNN
 F 1 "1k" V 1500 3700 50  0000 C CNN
-F 2 "" H 1500 3700 50  0001 C CNN
+F 2 "Resistors_SMD:R_0402" H 1500 3700 50  0001 C CNN
 F 3 "" H 1500 3700 50  0001 C CNN
 	1    1500 3700
@@
 $EndComp
 $Comp
-L R_Small R?
+L R_Small R30
 U 1 1 59461177
 P 1500 3600
-F 0 "R?" V 1550 3750 50  0000 C CNN
+F 0 "R30" V 1550 3750 50  0000 C CNN
 F 1 "1k" V 1500 3600 50  0000 C CNN
-F 2 "" H 1500 3600 50  0001 C CNN
+F 2 "Resistors_SMD:R_0402" H 1500 3600 50  0001 C CNN
 F 3 "" H 1500 3600 50  0001 C CNN
 	1    1500 3600
@@
 $EndComp
 $Comp
-L R_Small R?
+L R_Small R29
 U 1 1 5946117D
 P 1500 3500
-F 0 "R?" V 1550 3650 50  0000 C CNN
+F 0 "R29" V 1550 3650 50  0000 C CNN
 F 1 "1k" V 1500 3500 50  0000 C CNN
-F 2 "" H 1500 3500 50  0001 C CNN
+F 2 "Resistors_SMD:R_0402" H 1500 3500 50  0001 C CNN
 F 3 "" H 1500 3500 50  0001 C CNN
 	1    1500 3500
@@
 $EndComp
 $Comp
-L R_Small R?
+L R_Small R28
 U 1 1 59461183
 P 1500 3400
-F 0 "R?" V 1550 3550 50  0000 C CNN
+F 0 "R28" V 1550 3550 50  0000 C CNN
 F 1 "1k" V 1500 3400 50  0000 C CNN
-F 2 "" H 1500 3400 50  0001 C CNN
+F 2 "Resistors_SMD:R_0402" H 1500 3400 50  0001 C CNN
 F 3 "" H 1500 3400 50  0001 C CNN
 	1    1500 3400
@@
 $EndComp
 $Comp
-L R_Small R?
+L R_Small R27
 U 1 1 59461189
 P 1500 3300
-F 0 "R?" V 1550 3450 50  0000 C CNN
+F 0 "R27" V 1550 3450 50  0000 C CNN
 F 1 "1k" V 1500 3300 50  0000 C CNN
-F 2 "" H 1500 3300 50  0001 C CNN
+F 2 "Resistors_SMD:R_0402" H 1500 3300 50  0001 C CNN
 F 3 "" H 1500 3300 50  0001 C CNN
 	1    1500 3300
@@
 $EndComp
 $Comp
-L R_Small R?
+L R_Small R26
 U 1 1 5946118F
 P 1500 3200
-F 0 "R?" V 1550 3350 50  0000 C CNN
+F 0 "R26" V 1550 3350 50  0000 C CNN
 F 1 "1k" V 1500 3200 50  0000 C CNN
-F 2 "" H 1500 3200 50  0001 C CNN
+F 2 "Resistors_SMD:R_0402" H 1500 3200 50  0001 C CNN
 F 3 "" H 1500 3200 50  0001 C CNN
 	1    1500 3200
@@
 $EndComp
 $Comp
-L R_Small R?
+L R_Small R25
 U 1 1 59461195
 P 1500 3100
-F 0 "R?" V 1550 3250 50  0000 C CNN
+F 0 "R25" V 1550 3250 50  0000 C CNN
 F 1 "1k" V 1500 3100 50  0000 C CNN
-F 2 "" H 1500 3100 50  0001 C CNN
+F 2 "Resistors_SMD:R_0402" H 1500 3100 50  0001 C CNN
 F 3 "" H 1500 3100 50  0001 C CNN
 	1    1500 3100
@@
 $EndComp
 $Comp
-L R_Small R?
+L R_Small R24
 U 1 1 5946119B
 P 1500 3000
-F 0 "R?" V 1550 3150 50  0000 C CNN
+F 0 "R24" V 1550 3150 50  0000 C CNN
 F 1 "1k" V 1500 3000 50  0000 C CNN
-F 2 "" H 1500 3000 50  0001 C CNN
+F 2 "Resistors_SMD:R_0402" H 1500 3000 50  0001 C CNN
 F 3 "" H 1500 3000 50  0001 C CNN
 	1    1500 3000

Commit message: A massive bunch of former changes waiting to be committed.
Parts:
- R10, R13, R19, R20, R21, R22, R23, R24, R25, R26, R27, R28, R29, R30, R31, R9: symbol R_Small -> GhostSensorboard-rescue:R_Small-RESCUE-GhostSensorboard
- R12: symbol R -> GhostSensorboard-rescue:R-RESCUE-GhostSensorboard
- U1: symbol TCA9548ARGER -> NorBot:TCA9548ARGER
- U10, U11, U12, U13, U2, U3, U7, U8: symbol GP2Y0E02B -> NorBot:GP2Y0E02B
Changed lines of the file:
@@
-EESchema Schematic File Version 2
-LIBS:GhostSensorboard-rescue
-LIBS:power
-LIBS:device
-LIBS:transistors
-LIBS:conn
-LIBS:linear
-LIBS:regul
-LIBS:74xx
-LIBS:cmos4000
-LIBS:adc-dac
-LIBS:memory
-LIBS:xilinx
-LIBS:microcontrollers
-LIBS:dsp
-LIBS:microchip
-LIBS:analog_switches
-LIBS:motorola
-LIBS:texas
-LIBS:intel
-LIBS:audio
-LIBS:interface
-LIBS:digital-audio
-LIBS:philips
-LIBS:display
-LIBS:cypress
-LIBS:siliconi
-LIBS:opto
-LIBS:atmel
-LIBS:contrib
-LIBS:valves
-LIBS:NorBot
-LIBS:switches
+EESchema Schematic File Version 4
 LIBS:GhostSensorboard-cache
 EELAYER 26 0
@@
 $EndDescr
 $Comp
-L GP2Y0E02B U2
+L NorBot:GP2Y0E02B U2
 U 1 1 58C86DA1
 P 7850 2000
@@
 $EndComp
 $Comp
-L GP2Y0E02B U3
+L NorBot:GP2Y0E02B U3
 U 1 1 58C86E23
 P 7850 2750
@@
 $EndComp
 $Comp
-L GP2Y0E02B U7
+L NorBot:GP2Y0E02B U7
 U 1 1 58C86E59
 P 7850 3500
@@
 $EndComp
 $Comp
-L GP2Y0E02B U8
+L NorBot:GP2Y0E02B U8
 U 1 1 58C86EAD
 P 7850 4250
@@
 $EndComp
 $Comp
-L GP2Y0E02B U10
+L NorBot:GP2Y0E02B U10
 U 1 1 58C8705F
 P 9750 2000
@@
 $EndComp
 $Comp
-L GP2Y0E02B U11
+L NorBot:GP2Y0E02B U11
 U 1 1 58C87065
 P 9750 2750
@@
 $EndComp
 $Comp
-L GP2Y0E02B U12
+L NorBot:GP2Y0E02B U12
 U 1 1 58C8706B
 P 9750 3500
@@
 $EndComp
 $Comp
-L GP2Y0E02B U13
+L NorBot:GP2Y0E02B U13
 U 1 1 58C87071
 P 9750 4250
@@
 $EndComp
 $Comp
-L TCA9548ARGER U1
+L NorBot:TCA9548ARGER U1
 U 1 1 58C87BBF
 P 4700 2750
@@
 $EndComp
 $Comp
-L R R12
+L GhostSensorboard-rescue:R-RESCUE-GhostSensorboard R12
 U 1 1 58C88FA5
 P 3850 2500
@@
 $EndComp
 $Comp
-L GND #PWR043
+L GhostSensorboard-rescue:GND-RESCUE-GhostSensorboard #PWR043
 U 1 1 58C891DA
 P 4100 4000
@@
 	3850 2250 4200 2250
 $Comp
-L +3V3 #PWR044
+L GhostSensorboard-rescue:+3V3-RESCUE-GhostSensorboard #PWR044
 U 1 1 58C89F76
 P 3850 2100
@@
 	9150 4400 9300 4400
 $Comp
-L GND #PWR045
+L GhostSensorboard-rescue:GND-RESCUE-GhostSensorboard #PWR045
 U 1 1 58C9A570
 P 8350 2150
@@
 $EndComp
 $Comp
-L GND #PWR046
+L GhostSensorboard-rescue:GND-RESCUE-GhostSensorboard #PWR046
 U 1 1 58C9ABDE
 P 8350 2900
@@
 $EndComp
 $Comp
-L GND #PWR047
+L GhostSensorboard-rescue:GND-RESCUE-GhostSensorboard #PWR047
 U 1 1 58C9AC15
 P 8350 3650
@@
 $EndComp
 $Comp
-L GND #PWR048
+L GhostSensorboard-rescue:GND-RESCUE-GhostSensorboard #PWR048
 U 1 1 58C9AF22
 P 8350 4400
@@
 $EndComp
 $Comp
-L GND #PWR049
+L GhostSensorboard-rescue:GND-RESCUE-GhostSensorboard #PWR049
 U 1 1 58C9B715
 P 10250 2150
@@
 $EndComp
 $Comp
-L GND #PWR050
+L GhostSensorboard-rescue:GND-RESCUE-GhostSensorboard #PWR050
 U 1 1 58C9B74C
 P 10250 2900
@@
 $EndComp
 $Comp
-L GND #PWR051
+L GhostSensorboard-rescue:GND-RESCUE-GhostSensorboard #PWR051
 U 1 1 58C9B783
 P 10250 3650
@@
 $EndComp
 $Comp
-L GND #PWR052
+L GhostSensorboard-rescue:GND-RESCUE-GhostSensorboard #PWR052
 U 1 1 58C9B7BA
 P 10250 4400
@@
 	8250 4400 8350 4400
 $Comp
-L +3V3 #PWR053
+L GhostSensorboard-rescue:+3V3-RESCUE-GhostSensorboard #PWR053
 U 1 1 58C9DB9B
 P 7250 1850
@@
 $EndComp
 $Comp
-L +3V3 #PWR054
+L GhostSensorboard-rescue:+3V3-RESCUE-GhostSensorboard #PWR054
 U 1 1 58C9E117
 P 7250 2600
@@
 $EndComp
 $Comp
-L +3V3 #PWR055
+L GhostSensorboard-rescue:+3V3-RESCUE-GhostSensorboard #PWR055
 U 1 1 58C9E14E
 P 7250 3350
@@
 $EndComp
 $Comp
-L +3V3 #PWR056
+L GhostSensorboard-rescue:+3V3-RESCUE-GhostSensorboard #PWR056
 U 1 1 58C9E185
 P 7250 4100
@@
 $EndComp
 $Comp
-L +3V3 #PWR057
+L GhostSensorboard-rescue:+3V3-RESCUE-GhostSensorboard #PWR057
 U 1 1 58C9FCAA
 P 9100 1850
@@
 $EndComp
 $Comp
-L +3V3 #PWR058
+L GhostSensorboard-rescue:+3V3-RESCUE-GhostSensorboard #PWR058
 U 1 1 58C9FCE1
 P 9100 2600
@@
 $EndComp
 $Comp
-L +3V3 #PWR059
+L GhostSensorboard-rescue:+3V3-RESCUE-GhostSensorboard #PWR059
 U 1 1 58C9FD18
 P 9100 3350
@@
 $EndComp
 $Comp
-L +3V3 #PWR060
+L GhostSensorboard-rescue:+3V3-RESCUE-GhostSensorboard #PWR060
 U 1 1 58C9FD4F
 P 9100 4100
@@
 	1150 3700 1400 3700
 $Comp
-L +3V3 #PWR061
+L GhostSensorboard-rescue:+3V3-RESCUE-GhostSensorboard #PWR061
 U 1 1 58CA550D
 P 1900 2100
@@
 TCA9548ARGER I2C multiplexer\nI2C address: 0x70\nFarnell no: 269-0239
 $Comp
-L R_Small R23
+L GhostSensorboard-rescue:R_Small-RESCUE-GhostSensorboard R23
 U 1 1 5945CFBC
 P 1500 2900
@@
 $EndComp
 $Comp
-L R_Small R22
+L GhostSensorboard-rescue:R_Small-RESCUE-GhostSensorboard R22
 U 1 1 5945F8C2
 P 1500 2800
@@
 $EndComp
 $Comp
-L R_Small R21
+L GhostSensorboard-rescue:R_Small-RESCUE-GhostSensorboard R21
 U 1 1 5945F8EE
 P 1500 2700
@@
 $EndComp
 $Comp
-L R_Small R20
+L GhostSensorboard-rescue:R_Small-RESCUE-GhostSensorboard R20
 U 1 1 5945F91C
 P 1500 2600
@@
 $EndComp
 $Comp
-L R_Small R19
+L GhostSensorboard-rescue:R_Small-RESCUE-GhostSensorboard R19
 U 1 1 5945F950
 P 1500 2500
@@
 $EndComp
 $Comp
-L R_Small R13
+L GhostSensorboard-rescue:R_Small-RESCUE-GhostSensorboard R13
 U 1 1 5945F986
 P 1500 2400
@@
 $EndComp
 $Comp
-L R_Small R10
+L GhostSensorboard-rescue:R_Small-RESCUE-GhostSensorboard R10
 U 1 1 5945F9C4
 P 1500 2300
@@
 $EndComp
 $Comp
-L R_Small R9
+L GhostSensorboard-rescue:R_Small-RESCUE-GhostSensorboard R9
 U 1 1 5945F9FA
 P 1500 2200
@@
 $EndComp
 $Comp
-L R_Small R31
+L GhostSensorboard-rescue:R_Small-RESCUE-GhostSensorboard R31
 U 1 1 59461171
 P 1500 3700
@@
 $EndComp
 $Comp
-L R_Small R30
+L GhostSensorboard-rescue:R_Small-RESCUE-GhostSensorboard R30
 U 1 1 59461177
 P 1500 3600
@@
 $EndComp
 $Comp
-L R_Small R29
+L GhostSensorboard-rescue:R_Small-RESCUE-GhostSensorboard R29
 U 1 1 5946117D
 P 1500 3500
@@
 $EndComp
 $Comp
-L R_Small R28
+L GhostSensorboard-rescue:R_Small-RESCUE-GhostSensorboard R28
 U 1 1 59461183
 P 1500 3400
@@
 $EndComp
 $Comp
-L R_Small R27
+L GhostSensorboard-rescue:R_Small-RESCUE-GhostSensorboard R27
 U 1 1 59461189
 P 1500 3300
@@
 $EndComp
 $Comp
-L R_Small R26
+L GhostSensorboard-rescue:R_Small-RESCUE-GhostSensorboard R26
 U 1 1 5946118F
 P 1500 3200
@@
 $EndComp
 $Comp
-L R_Small R25
+L GhostSensorboard-rescue:R_Small-RESCUE-GhostSensorboard R25
 U 1 1 59461195
 P 1500 3100
@@
 $EndComp
 $Comp
-L R_Small R24
+L GhostSensorboard-rescue:R_Small-RESCUE-GhostSensorboard R24
 U 1 1 5946119B
 P 1500 3000
