File: KiCad/GhostESP32/Rev4/GhostESP32.sch (KiCad schematic (older format))
At the start: 50 parts, among them J1 USB_OTG, J2 CONN_01X12, J3 CONN_01X12, J4 STEERING, J5 MOTOR, Q1 Q_NPN_BEC, Q2 Q_NPN_BEC, Q3 Q_NPN_BEC, Q4 BSS138, Q5 BSS138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

Commit message: A massive bunch of former changes waiting to be committed.
Parts:
- added U6, U7: NeoPixelNano, NorBotKiCadFootprints:NeoPixelNano, symbol NorBot:NeoPixelNano
- C1, C10, C11, C12, C2, C3, C4, C5, C6, C7, C8, C9: symbol C_Small -> GhostESP32-rescue:C_Small-RESCUE-GhostESP32
- D1, D2, D3, D4, D5: symbol D_Zener_Small_ALT -> GhostESP32-rescue:D_Zener_Small_ALT-RESCUE-GhostESP32
- D6, D7: symbol LED_ALT -> GhostESP32-rescue:LED_ALT-RESCUE-GhostESP32
- J1: symbol USB_OTG -> GhostESP32-rescue:USB_OTG-RESCUE-GhostESP32
- J2, J3: symbol CONN_01X12 -> GhostESP32-rescue:CONN_01X12-RESCUE-GhostESP32
- J4, J5: symbol CONN_01X03 -> GhostESP32-rescue:CONN_01X03-RESCUE-GhostESP32
- Q1, Q2, Q3: symbol Q_NPN_BEC -> GhostESP32-rescue:Q_NPN_BEC-RESCUE-GhostESP32
- Q4, Q5: symbol BSS138 -> GhostESP32-rescue:BSS138-RESCUE-GhostESP32
- R1, R10, R11, R12, R13, R14, R15, R2, R3, R4, R5, R6, R7, R8, R9: symbol R_Small -> GhostESP32-rescue:R_Small-RESCUE-GhostESP32
- SW1: symbol SW_SPDT -> GhostESP32-rescue:SW_SPDT-RESCUE-GhostESP32
- U1: symbol NCP1117-3.3_SOT223 -> GhostESP32-rescue:NCP1117-3.3_SOT223-RESCUE-GhostESP32
- U2: symbol CP2102 -> NorBot:CP2102
- U3: symbol TMP102 -> NorBot:TMP102
- U4: symbol MPU-9250 -> NorBot:MPU-9250
- U5: symbol ESP-WROOM-32 -> NorBot:ESP-WROOM-32
Connections:
- net labels added: NEOPIXEL
- wire segments 186 -> 231
- no-connect marks 23 -> 24
Other:
- note added: "Nexpixel leds\nAdafruit prod no: 3484"
- moved on the sheet: C12, R15, SW1
