File: KiCad/GhostESP32/Rev5/GhostESP32.kicad_pcb (KiCad board)
At the start: 2 copper layers, 76.7 x 56.7 mm, 52 parts, among them J1 USB_OTG, J2 CONN_01X12, J3 CONN_01X12, J4 STEERING, J5 MOTOR, Q1 Q_NPN_BEC, Q2 Q_NPN_BEC, Q3 Q_NPN_BEC, Q4 BSS138, Q5 BSS138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

Commit message: Started on Rev5 of GhostESP32
Parts:
- U3: footprint TO_SOT_Packages_SMD:SOT-23-6 -> NorBotKiCadFootprints:SOT563
Connections:
- J1 pad 4: Net-(J1-Pad4) -> (no net)
- SW1 pad 1: Net-(SW1-Pad1) -> (no net)
- U2 pad 1: Net-(U2-Pad1) -> (no net)
- U2 pad 10: Net-(U2-Pad10) -> (no net)
- U2 pad 11: Net-(U2-Pad11) -> (no net)
- U2 pad 12: Net-(U2-Pad12) -> (no net)
- U2 pad 13: Net-(U2-Pad13) -> (no net)
- U2 pad 14: Net-(U2-Pad14) -> (no net)
- U2 pad 15: Net-(U2-Pad15) -> (no net)
- U2 pad 16: Net-(U2-Pad16) -> (no net)
- U2 pad 17: Net-(U2-Pad17) -> (no net)
- U2 pad 18: Net-(U2-Pad18) -> (no net)
- U2 pad 19: Net-(U2-Pad19) -> (no net)
- U2 pad 2: Net-(U2-Pad2) -> (no net)
- U2 pad 20: Net-(U2-Pad20) -> (no net)
- U2 pad 21: Net-(U2-Pad21) -> (no net)
- U2 pad 22: Net-(U2-Pad22) -> (no net)
- U2 pad 23: Net-(U2-Pad23) -> (no net)
- U2 pad 27: Net-(U2-Pad27) -> (no net)
- U2 pad 9: Net-(U2-Pad9) -> (no net)
- U4 pad 19: Net-(U4-Pad19) -> (no net)
- U4 pad 21: Net-(U4-Pad21) -> (no net)
- U4 pad 7: Net-(U4-Pad7) -> (no net)
- U5 pad 14: IO12 -> (no net)
- U5 pad 17: Net-(U5-Pad17) -> (no net)
- U5 pad 18: Net-(U5-Pad18) -> (no net)
- U5 pad 19: Net-(U5-Pad19) -> (no net)
- U5 pad 20: Net-(U5-Pad20) -> (no net)
- U5 pad 21: Net-(U5-Pad21) -> (no net)
- U5 pad 22: Net-(U5-Pad22) -> (no net)
- U5 pad 23: IO15 -> (no net)
- U5 pad 24: IO2 -> (no net)
- U5 pad 29: IO5 -> (no net)
- U5 pad 32: Net-(U5-Pad32) -> (no net)
- U6 pad 3: NEOPIXEL -> (no net)
- U7 pad 1: Net-(U7-Pad1) -> (no net)
Routing:
- net IO33/SDA: track 71.8 -> 72.6 mm
- net +3V3: track 217.1 -> 217.9 mm
- net GND: track 182.4 -> 181.8 mm
Other:
- board text added: "Ghost32 Rev 5 Frode Lillerud 9.feb 2018"
- board text removed: "Ghost32 Rev 4 Frode Lillerud 23.aug 2017"
