File: KiCad/GhostESP32/Rev5/GhostESP32.sch (KiCad schematic (older format))
At the start: 52 parts, among them J1 USB_OTG, J2 CONN_01X12, J3 CONN_01X12, J4 STEERING, J5 MOTOR, Q1 Q_NPN_BEC, Q2 Q_NPN_BEC, Q3 Q_NPN_BEC, Q4 BSS138, Q5 BSS138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

Commit message: Working on revision 5 of the PCBs
Parts:
- removed U6, U7: NeoPixelNano, NorBotKiCadFootprints:NeoPixelNano, symbol NorBot:NeoPixelNano
- R13, R14: value 2k2 -> 10k
Connections:
- net labels added: IO21(SDA), IO22(SCL), IO32, IO33
- net labels removed: IO21, IO22, IO32/SCL, IO33/SDA, NEOPIXEL
- wire segments 231 -> 222
- no-connect marks 24 -> 23
Other:
- note added: "Board powered by 5V either via USB, or from ESC connected to motor headers.\nNote, GPIO 34-39 are INPUT mode ONLY\nNote, GPIO 6-11 are used by SPI-flash, and canot be used for other purposes\nNote, GPIO0, GPIO2, GPIO5, GPIO12 and GPIO15 are strapping pins, and cannot be pulled high/low.\nNote, GPIO23 is dedicated to LED\nNote, GPIO21 (SDA) and GPIO22 (SCL) are dedicated to I2C"
- note added: "I2C pullups\nUse range 2k2 - 10k"
- note removed: "Board powered by 5V either via USB, or from ESC connected to motor headers.\nNote, GPIO 34-39 are INPUT mode ONLY\nNote, GPIO 6-11 are used by SPI-flash, and canot be used for other purposes\nNote, GPIO0, GPIO2, GPIO5, GPIO12 and GPIO15 are strapping pins, and cannot be pulled high/low.\nNote, GPIO23 is dedicated to LED\nNote, GPIO32 and GPIO33 are dedicated to I2C"
- note removed: "I2C pullups"
- note removed: "Nexpixel leds\nAdafruit prod no: 3484"
- moved on the sheet: C1, C12, C2, D4, D5, D6, D7, Q3, R13, R14, R15, R5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
