File: KiCad/GhostSensorboard/Rev5/GhostSensorBoard/GhostSensorBoard.kicad_pcb (KiCad board)
At the start: 2 copper layers, 70 x 43 mm, 0 parts

Commit message: Rev 5 of boards sent to production
Parts:
- added C1: 1nF, Capacitor_SMD:C_0603_1608Metric, F.Cu at (172.2, 92.7)
- added C2: 2.2uF - 10uF, Capacitor_SMD:C_0603_1608Metric, F.Cu at (136.8, 98.4)
- added D1: LED, LED_SMD:LED_0603_1608Metric, F.Cu at (127.4, 117.5)
- added D2: LED, LED_SMD:LED_0603_1608Metric, F.Cu at (127.1, 85.0)
- added D3: LED, LED_SMD:LED_0603_1608Metric, F.Cu at (179.5, 114.5)
- added D4: LED, LED_SMD:LED_0603_1608Metric, F.Cu at (180.4, 85.4)
- added J1: Li-Po BATTERY, Connector_PinHeader_2.54mm:PinHeader_1x02_P2.54mm_Vertical, F.Cu at (144.6, 119.0)
- added J2: Conn_01x03, Connector_PinHeader_2.54mm:PinHeader_1x03_P2.54mm_Vertical, F.Cu at (151.0, 88.1)
- added J3: Conn_01x12, Connector_PinHeader_2.54mm:PinHeader_1x12_P2.54mm_Vertical, F.Cu at (151.0, 80.4)
- added J4: Conn_01x12, Connector_PinHeader_2.54mm:PinHeader_1x12_P2.54mm_Vertical, F.Cu at (151.0, 119.0)
- added R1: 2k2, Resistor_SMD:R_0402_1005Metric, F.Cu at (146.3, 96.0)
- added R10: 1k, Resistor_SMD:R_0402_1005Metric, F.Cu at (180.7, 108.5)
- added R11: 1k, Resistor_SMD:R_0402_1005Metric, F.Cu at (180.8, 106.9)
- added R12: 1k, Resistor_SMD:R_0402_1005Metric, F.Cu at (180.3, 100.5)
- added R13: 1k, Resistor_SMD:R_0402_1005Metric, F.Cu at (180.3, 98.5)
- added R14: 1k, Resistor_SMD:R_0402_1005Metric, F.Cu at (180.5, 91.4)
- added R15: 1k, Resistor_SMD:R_0402_1005Metric, F.Cu at (180.6, 89.8)
- added R16: 1k, Resistor_SMD:R_0402_1005Metric, F.Cu at (142.2, 85.7)
- added R17: 1k, Resistor_SMD:R_0402_1005Metric, F.Cu at (140.8, 85.6)
- added R18: 330, Resistor_SMD:R_0402_1005Metric, F.Cu at (131.9, 117.5)
- added R19: 330, Resistor_SMD:R_0402_1005Metric, F.Cu at (126.8, 81.5)
- added R2: 1k, Resistor_SMD:R_0402_1005Metric, F.Cu at (133.2, 86.2)
- added R20: 330, Resistor_SMD:R_0402_1005Metric, F.Cu at (178.9, 112.7)
- added R21: 330, Resistor_SMD:R_0402_1005Metric, F.Cu at (183.8, 85.6)
- added R22: 470, Resistor_SMD:R_0402_1005Metric, F.Cu at (165.6, 88.3)
- added R23: 270, Resistor_SMD:R_0402_1005Metric, F.Cu at (151.3, 114.4)
- added R24: 10k, Resistor_SMD:R_0402_1005Metric, F.Cu at (156.3, 114.2)
- added R3: 1k, Resistor_SMD:R_0402_1005Metric, F.Cu at (131.2, 86.1)
- added R4: 1k, Resistor_SMD:R_0402_1005Metric, F.Cu at (127.0, 93.0)
- added R5: 1k, Resistor_SMD:R_0402_1005Metric, F.Cu at (127.0, 94.5)
- added R6: 1k, Resistor_SMD:R_0402_1005Metric, F.Cu at (128.0, 100.0)
- added R7: 1k, Resistor_SMD:R_0402_1005Metric, F.Cu at (128.1, 102.2)
- added R8: 1k, Resistor_SMD:R_0402_1005Metric, F.Cu at (126.6, 109.2)
- added R9: 1k, Resistor_SMD:R_0402_1005Metric, F.Cu at (126.6, 110.5)
- added SW1: SW_Push, Button_Switch_SMD:SW_SPST_EVQP2, F.Cu at (165.6, 92.6)
- added SW2: SW_SPDT, NorBotKiCadFootprints:MFP106D, F.Cu at (136.5, 110.7)
- added U1: TCA9548APWR, Package_SO:TSSOP-24_4.4x7.8mm_P0.65mm, F.Cu at (152.9, 98.8)
- added U10: Transmissive_Photo_Interrupter, Connector_PinHeader_2.54mm:PinHeader_1x04_P2.54mm_Vertical, F.Cu at (151.2, 110.2)
- added U11: TMP102, Package_TO_SOT_SMD:SOT-23-6, F.Cu at (167.3, 103.0)
- added U12: MIC5219-5.0, Package_TO_SOT_SMD:SOT-23-5, F.Cu at (136.8, 103.0)
- added U2: GP2Y0E02B, Connector_JST:JST_SH_BM04B-SRSS-TB_1x04_P1.00mm_Vertical, F.Cu at (132.8, 81.3)
- added U3: GP2Y0E02B, Connector_JST:JST_SH_BM04B-SRSS-TB_1x04_P1.00mm_Vertical, F.Cu at (121.9, 92.5)
- added U4: GP2Y0E02B, Connector_JST:JST_SH_BM04B-SRSS-TB_1x04_P1.00mm_Vertical, F.Cu at (122.0, 100.9)
- added U5: GP2Y0E02B, Connector_JST:JST_SH_BM04B-SRSS-TB_1x04_P1.00mm_Vertical, F.Cu at (122.0, 109.0)
- added U6: GP2Y0E02B, Connector_JST:JST_SH_BM04B-SRSS-TB_1x04_P1.00mm_Vertical, F.Cu at (185.9, 108.4)
- added U7: GP2Y0E02B, Connector_JST:JST_SH_BM04B-SRSS-TB_1x04_P1.00mm_Vertical, F.Cu at (185.8, 100.0)
- added U8: GP2Y0E02B, Connector_JST:JST_SH_BM04B-SRSS-TB_1x04_P1.00mm_Vertical, F.Cu at (185.8, 91.3)
- added U9: GP2Y0E02B, Connector_JST:JST_SH_BM04B-SRSS-TB_1x04_P1.00mm_Vertical, F.Cu at (142.3, 81.3)
Routing:
- net +3V3: track 0.00 -> 280.4 mm, vias 0 -> 15
- net GND: track 0.00 -> 141.7 mm, vias 0 -> 9
- net LED: track 0.00 -> 122.5 mm, vias 0 -> 4
- net BUTTON: track 0.00 -> 48.6 mm, vias 0 -> 1
- net +5V: track 0.00 -> 36.6 mm, vias 0 -> 3
- net IO22(SCL): track 0.00 -> 36.6 mm, vias 0 -> 2
- net IO21(SDA): track 0.00 -> 36.2 mm, vias 0 -> 2
- net SC6: track 0.00 -> 33.4 mm, vias 0 -> 2
- net SC4: track 0.00 -> 33.2 mm
- net SD4: track 0.00 -> 32.8 mm
- net SD6: track 0.00 -> 32.7 mm, vias 0 -> 2
- net SC3: track 0.00 -> 31.3 mm
- net SD5: track 0.00 -> 30.7 mm, vias 0 -> 2
- net SD3: track 0.00 -> 30.6 mm
- net SD1: track 0.00 -> 30.4 mm
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- added copper zone on B.Cu, net GND
- added copper zone on F.Cu, net GND
Other:
- net class POWER added: clearance 0.2, trace_width 0.35, via_dia 0.8, via_drill 0.4
- board text added: "+"
- board text added: "+3V3"
- board text added: "+5V"
- board text added: "-"
- board text added: "3V3"
- board text added: "BUTTON"
- board text added: "ENCODER"
- board text added: "GND"
- board text added: "Ghost Sensorboard, Rev 5 Frode Lillerud 18.mar 2018"
- board text added: "I36"
- board text added: "IO13"
- board text added: "IO21(SDA)"
- board text added: "IO22(SCL)"
- board text added: "IO25"
- board text added: "LED"
- board text added: "LiPo (5V-12V)"
- board text added: "OFF"
- board text added: "ON"
- board text added: "SM_SIG"
- board text added: "SM_VCC"
