File: KiCad/GhostSensorboard/Rev5/GhostSensorBoard/GhostSensorBoard.sch (KiCad schematic (older format))
At the start: 48 parts, among them J1 Conn_01x12, J2 Conn_01x03, J3 Conn_01x12, U1 TCA9548APWR, U2 GP2Y0E02B

Commit message: Rev 5 of boards sent to production
Parts:
- C1, C2: renamed from C?; footprint (none) -> Capacitor_SMD:C_0603_1608Metric
- D1, D2, D3, D4: renamed from D?; footprint (none) -> LED_SMD:LED_0603_1608Metric
- J1: renamed from J?; footprint (none) -> Connector_PinHeader_2.54mm:PinHeader_1x02_P2.54mm_Vertical
- J2: footprint (none) -> Connector_PinHeader_2.54mm:PinHeader_1x03_P2.54mm_Vertical
- J3: renamed from J1; footprint (none) -> Connector_PinHeader_2.54mm:PinHeader_1x12_P2.54mm_Vertical
- J4: renamed from J3; footprint (none) -> Connector_PinHeader_2.54mm:PinHeader_1x12_P2.54mm_Vertical
- R1, R18, R19, R20, R21, R22, R23, R24: renamed from R?; footprint (none) -> Resistor_SMD:R_0402_1005Metric
- R10: renamed from R9; footprint (none) -> Resistor_SMD:R_0402_1005Metric
- R11: renamed from R10; footprint (none) -> Resistor_SMD:R_0402_1005Metric
- R12: renamed from R11; footprint (none) -> Resistor_SMD:R_0402_1005Metric
- R13: renamed from R12; footprint (none) -> Resistor_SMD:R_0402_1005Metric
- R14: renamed from R13; footprint (none) -> Resistor_SMD:R_0402_1005Metric
- R15: renamed from R14; footprint (none) -> Resistor_SMD:R_0402_1005Metric
- R16: renamed from R15; footprint (none) -> Resistor_SMD:R_0402_1005Metric
- R17: renamed from R16; footprint (none) -> Resistor_SMD:R_0402_1005Metric
- R2: renamed from R1; footprint (none) -> Resistor_SMD:R_0402_1005Metric
- R3: renamed from R2; footprint (none) -> Resistor_SMD:R_0402_1005Metric
- R4: renamed from R3; footprint (none) -> Resistor_SMD:R_0402_1005Metric
- R5: renamed from R4; footprint (none) -> Resistor_SMD:R_0402_1005Metric
- R6: renamed from R5; footprint (none) -> Resistor_SMD:R_0402_1005Metric
- R7: renamed from R6; footprint (none) -> Resistor_SMD:R_0402_1005Metric
- R8: renamed from R7; footprint (none) -> Resistor_SMD:R_0402_1005Metric
- R9: renamed from R8; footprint (none) -> Resistor_SMD:R_0402_1005Metric
- SW1: renamed from SW?; footprint (none) -> Button_Switch_SMD:SW_SPST_EVQP2
- SW2: renamed from SW?; footprint (none) -> NorBotKiCadFootprints:MFP106D
- U1: footprint (none) -> Package_SO:TSSOP-24_4.4x7.8mm_P0.65mm
- U10: renamed from U?; footprint (none) -> Connector_PinHeader_2.54mm:PinHeader_1x04_P2.54mm_Vertical
- U11: renamed from U?; footprint TO_SOT_Packages_SMD:SOT-23-6 -> Package_TO_SOT_SMD:SOT-23-6
- U2: footprint (none) -> Connector_JST:JST_SH_BM04B-SRSS-TB_1x04_P1.00mm_Vertical
- U3, U4, U5, U6, U7, U8, U9: renamed from U?; footprint (none) -> Connector_JST:JST_SH_BM04B-SRSS-TB_1x04_P1.00mm_Vertical
- gave numbers to parts that had none: 1
Connections:
- net IO13: now also J2.1 (Pin_1)
- net IO17: no longer J2.1 (Pin_1)
- no-connect marks 2 -> 12
